File: GR-LRR-PCB/GR-LRR-PCB.kicad_sch (KiCad schematic)
At the start: 0 parts

Commit message: selected parts for power side
Other:
- added sheet Control (Control.kicad_sch)
- added sheet IO (IO.kicad_sch)
- added sheet PowerSystem (PowerSystem.kicad_sch)
- note added: "1. Motor Drivers 2. H7 Mount 3. 24v to 5v 4. 5v to 3.3v 5. UT 6. Motor Wire mount 7. Relay mount 8. clamp sensor 9. encoder 10. linear transducer 11. Hard estop 12. main battery power in 13. Battery Monitor"
- note removed: "1. Motor Drivers 2. H7 Mount"
Changed lines of the file:
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@@
 (kicad_sch (version 20230121) (generator eeschema)
-  (paper "A4")
-  (text "1. Motor Drivers\n2. H7 Mount" (at 29.21 36.83 0)
+  (paper "A")
+  (text "1. Motor Drivers\n2. H7 Mount\n3. 24v to 5v\n4. 5v to 3.3v\n5. UT\n6. Motor Wire mount\n7. Relay mount\n8. clamp sensor\n9. encoder\n10. linear transducer\n11. Hard estop\n12. main battery power in\n13. Battery Monitor"
+    (at 24.13 90.17 0)
     (effects (font (size 1.27 1.27)) (justify left bottom))
   )
+  (sheet (at 50.8 20.32) (size 31.75 25.4) (fields_autoplaced)
+    (stroke (width 0.1524) (type solid))
+    (fill (color 0 0 0 0.0000))
+    (property "Sheetname" "IO" (at 50.8 19.6084 0)
+      (effects (font (size 1.27 1.27)) (justify left bottom))
+    )
+    (property "Sheetfile" "IO.kicad_sch" (at 50.8 46.3046 0)
+      (effects (font (size 1.27 1.27)) (justify left top))
+    )
+    (instances
+      (project "GR-LRR-PCB"
+        (path "/f2632f9f-3f36-4af8-bf53-b0ff2066ae87" (page "3"))
+      )
+    )
+  )
+  (sheet (at 86.36 20.32) (size 31.75 25.4) (fields_autoplaced)
+    (stroke (width 0.1524) (type solid))
+    (fill (color 0 0 0 0.0000))
+    (property "Sheetname" "Control" (at 86.36 19.6084 0)
+      (effects (font (size 1.27 1.27)) (justify left bottom))
+    )
+    (property "Sheetfile" "Control.kicad_sch" (at 86.36 46.3046 0)
+      (effects (font (size 1.27 1.27)) (justify left top))
+    )
+    (instances
+      (project "GR-LRR-PCB"
+        (path "/f2632f9f-3f36-4af8-bf53-b0ff2066ae87" (page "4"))
+      )
+    )
+  )
+  (sheet (at 15.24 20.32) (size 30.48 25.4) (fields_autoplaced)
+    (stroke (width 0.1524) (type solid))
+    (fill (color 0 0 0 0.0000))
+    (property "Sheetname" "PowerSystem" (at 15.24 19.6084 0)
+      (effects (font (size 1.27 1.27)) (justify left bottom))
+    )
+    (property "Sheetfile" "PowerSystem.kicad_sch" (at 15.24 46.3046 0)
+      (effects (font (size 1.27 1.27)) (justify left top))
+    )
+    (instances
+      (project "GR-LRR-PCB"
+        (path "/f2632f9f-3f36-4af8-bf53-b0ff2066ae87" (page "2"))
+      )
+    )
+  )
   (sheet_instances

Commit message: starting first layout
Other:
- sheet Control renamed Controller
- sheet Controller: file Control.kicad_sch -> Controller.kicad_sch
Changed lines of the file:
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@@
     (stroke (width 0.1524) (type solid))
     (fill (color 0 0 0 0.0000))
-    (property "Sheetname" "Control" (at 86.36 19.6084 0)
+    (property "Sheetname" "Controller" (at 86.36 19.6084 0)
       (effects (font (size 1.27 1.27)) (justify left bottom))
     )
-    (property "Sheetfile" "Control.kicad_sch" (at 86.36 46.3046 0)
+    (property "Sheetfile" "Controller.kicad_sch" (at 86.36 46.3046 0)
       (effects (font (size 1.27 1.27)) (justify left top))
     )
