File: GR-LRR-CONTROL-PCB/GR-LRR-CONTROL-PCB.kicad_pcb (KiCad board)
At the start: 2 copper layers, 143.9 x 92.9 mm, 25 parts, among them IC1 MC1413DR2G, J1 DRIVER 1, J10 FX30B-4S-3.81DSA, J11 FX30B-4S-3.81DSA, J2 DRIVER 3, J3 DRIVER 2, J4 DRIVER 4, J5 LED, J6 CLAMP, J7 UT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

Commit message: save
Parts:
- added LED1: QTLP650C2TR, QTLP650C2TR:LEDC3216X130N, F.Cu at (143.6, 115.2)
- added LED2: QTLP650C2TR, QTLP650C2TR:LEDC3216X130N, F.Cu at (167.2, 85.7)
- added LED4: QTLP650C2TR, QTLP650C2TR:LEDC3216X130N, F.Cu at (175.8, 112.6)
- added LED5: QTLP650C2TR, QTLP650C2TR:LEDC3216X130N, F.Cu at (175.8, 117.4)
- added LED6: QTLP650C2TR, QTLP650C2TR:LEDC3216X130N, F.Cu at (175.8, 122.0)
- added R10: 1200ohm, 0.5w, Resistor_SMD:R_1206_3216Metric_Pad1.30x1.75mm_HandSolder, F.Cu at (181.1, 112.6)
- added R11: 180ohm, 1/10w, Resistor_SMD:R_1206_3216Metric_Pad1.30x1.75mm_HandSolder, F.Cu at (181.1, 117.4)
- added R12: 75ohm, 1/10w, Resistor_SMD:R_1206_3216Metric_Pad1.30x1.75mm_HandSolder, F.Cu at (181.1, 121.2)
- added R13: 10k, Resistor_SMD:R_1206_3216Metric_Pad1.30x1.75mm_HandSolder, F.Cu at (113.8, 124.0)
- added R14: 10k, Resistor_SMD:R_1206_3216Metric_Pad1.30x1.75mm_HandSolder, F.Cu at (113.8, 120.1)
- added R7: 75ohm, 1/10w, Resistor_SMD:R_1206_3216Metric_Pad1.30x1.75mm_HandSolder, F.Cu at (143.6, 120.5)
- added R8: 10k, Resistor_SMD:R_1206_3216Metric_Pad1.30x1.75mm_HandSolder, F.Cu at (113.8, 128.0)
- added R9: 75ohm, 1/10w, Resistor_SMD:R_1206_3216Metric_Pad1.30x1.75mm_HandSolder, F.Cu at (161.9, 85.7)
- IC1: moved to F.Cu
- moved R6 54.5 mm to (156.5, 85.7), turned to 180 degrees
- moved Q1 53.0 mm to (159.3, 94.3), turned to 90 degrees
- moved Q2 52.3 mm to (164.9, 94.3), turned to 90 degrees
- moved IC1 6.49 mm to (121.4, 124.2), turned to 180 degrees
- moved R5 5.09 mm to (169.5, 73.5)
- moved R4 5.09 mm to (169.5, 67.9)
- moved U2 1.72 mm to (159.0, 116.2)
Connections:
- net DO STEPPER ENABLE renamed D0 STEPPER ENABLE
- DR1 pad 4: unconnected-(DR1-STEP/AIN1-Pad4) -> D1 STEP 1
- DR1 pad 5: unconnected-(DR1-DIR/AIN2-Pad5) -> GPIO0 DIR 1
- DR2 pad 4: unconnected-(DR2-STEP/AIN1-Pad4) -> D2 STEP 2
- DR2 pad 5: unconnected-(DR2-DIR/AIN2-Pad5) -> GPIO1 DIR 2
- DR3 pad 4: unconnected-(DR3-STEP/AIN1-Pad4) -> D3 STEP 3
- DR3 pad 5: unconnected-(DR3-DIR/AIN2-Pad5) -> GPIO2 DIR 3
- DR4 pad 4: unconnected-(DR4-STEP/AIN1-Pad4) -> D4 STEP 4
- DR4 pad 5: unconnected-(DR4-DIR/AIN2-Pad5) -> GPIO3 DIR 4
- IC1 pad 1: 50_GPIO2_PD4 -> GPIO4 RED LED
- IC1 pad 2: 48_GPIO1_PC15 -> GPIO5 YELLOW LED
- IC1 pad 3: 46_GPIO0_PC13 -> GPIO6 GREEN LED
- J5 pad 2: Net-(IC1-OUT_7) -> Net-(J5-Pad2)
- J5 pad 3: Net-(IC1-OUT_6) -> Net-(J5-Pad3)
- J5 pad 4: Net-(IC1-OUT_5) -> Net-(J5-Pad4)
- J6 pad 1: 52_GPIO3_PD5 -> D5 CLAMP
- R1 pad 2: 52_GPIO3_PD5 -> D5 CLAMP
- U1 pad J1_21: Net-(U1A-VIN-PadJ1_21) -> +5V
- U1 pad J1_22: Net-(U1A-GND-PadJ1_22) -> GND
- U1 pad J1_31: Net-(U1A-GND-PadJ1_22) -> Net-(U1A-GND-PadJ1_31)
- U1 pad J1_32: Net-(U1A-VIN-PadJ1_21) -> unconnected-(U1A-VIN-PadJ1_32)
- U1 pad J1_41: Net-(U1A-VIN-PadJ1_21) -> +5V
- U1 pad J1_42: Net-(U1A-GND-PadJ1_22) -> GND
- U1 pad J1_47: Net-(U1A-GND-PadJ1_22) -> Net-(U1A-GND-PadJ1_31)
- U1 pad J1_48: Net-(U1A-VIN-PadJ1_21) -> unconnected-(U1A-VIN-PadJ1_48)
- U1 pad J1_54: Net-(U1A-GND-PadJ1_22) -> Net-(U1A-GND-PadJ1_31)
- U1 pad J2_23: Net-(U1B-VCC/+3V3-PadJ2_23) -> unconnected-(U1B-VCC/+3V3-PadJ2_23)
- U1 pad J2_24: Net-(U1B-GND_1-PadJ2_24) -> GND
- U1 pad J2_33: Net-(U1B-GND_1-PadJ2_24) -> GND
- U1 pad J2_43: Net-(U1B-VCC/+3V3-PadJ2_23) -> unconnected-(U1B-VCC/+3V3-PadJ2_43)
- U1 pad J2_44: Net-(U1B-GND_1-PadJ2_24) -> GND
- U1 pad J2_46: unconnected-(U1B-GPIO_0-PadJ2_46) -> GPIO0 DIR 1
- U1 pad J2_48: unconnected-(U1B-GPIO_1-PadJ2_48) -> GPIO1 DIR 2
- U1 pad J2_50: unconnected-(U1B-GPIO_2-PadJ2_50) -> GPIO2 DIR 3
- U1 pad J2_52: unconnected-(U1B-GPIO_3-PadJ2_52) -> GPIO3 DIR 4
- U1 pad J2_54: unconnected-(U1B-GPIO_4-PadJ2_54) -> GPIO4 RED LED
- U1 pad J2_56: unconnected-(U1B-GPIO_5-PadJ2_56) -> GPIO5 YELLOW LED
- U1 pad J2_57: Net-(U1B-GND_1-PadJ2_24) -> GND
- U1 pad J2_58: unconnected-(U1B-GPIO_6-PadJ2_58) -> GPIO6 GREEN LED
- U1 pad J2_60: unconnected-(U1B-PWM_6-PadJ2_60) -> D1 STEP 1
- U1 pad J2_61: unconnected-(U1B-PWM_2-PadJ2_61) -> D5 CLAMP
- U1 pad J2_63: unconnected-(U1B-PWM_3-PadJ2_63) -> D4 STEP 4
- U1 pad J2_65: unconnected-(U1B-PWM_4-PadJ2_65) -> D3 STEP 3
- U1 pad J2_67: unconnected-(U1B-PWM_5-PadJ2_67) -> D2 STEP 2
- U1 pad J2_69: Net-(U1B-VCC/+3V3-PadJ2_23) -> unconnected-(U1B-VCC/+3V3-PadJ2_69)
- U1 pad J2_70: Net-(U1B-GND_1-PadJ2_24) -> GND
- U2 pad 1: unconnected-(U2-VCC-Pad1) -> +3.3V
Routing:
- net +3.3V: track 0.00 -> 338.6 mm, vias 0 -> 5
- net +5V: track 0.00 -> 238.1 mm, vias 0 -> 1
- net +24V: track 0.00 -> 187.9 mm, vias 0 -> 2
- net D10 CIPO: track 0.00 -> 145.5 mm, vias 0 -> 2
- net D8 COPI: track 0.00 -> 141.8 mm, vias 0 -> 5
- net D9 CK: track 0.00 -> 136.8 mm, vias 0 -> 10
- net D7 CS: track 0.00 -> 128.6 mm, vias 0 -> 11
- net STEPPER_ENABLE: track 0.00 -> 128.4 mm, vias 0 -> 14
- net 73_ANALOG_A0: track 0.00 -> 89.0 mm, vias 0 -> 2
- net GPIO0 DIR 1: track 0.00 -> 86.0 mm, vias 0 -> 2
- net D1 STEP 1: track 0.00 -> 83.3 mm
- net D4 STEP 4: track 0.00 -> 80.2 mm
- net D0 STEPPER ENABLE: track 0.00 -> 79.5 mm, vias 0 -> 2
- net 75_ANALOG_A1: track 0.00 -> 71.4 mm, vias 0 -> 2
- net GPIO4 RED LED: track 0.00 -> 62.0 mm
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- added copper zone on B.Cu, net +24V
- added copper zone on B.Cu, net GND
- added copper zone on F.Cu, net GND
Other:
- board text added: "GR-LRR-CONTROL-A1 12072023"
