File: GR-LRR-CONTROL-PCB/GR-LRR-CONTROL-PCB.kicad_sch (KiCad schematic)
At the start: 25 parts, among them IC1 MC1413DR2G, J1 DRIVER 1, J10 FX30B-4S-3.81DSA, J11 FX30B-4S-3.81DSA, J2 DRIVER 3, J3 DRIVER 2, J4 DRIVER 4, J5 LED, J6 CLAMP, J7 UT, Q1 BSS806NH6327XTSA1, Q2 BSS806NH6327XTSA1, SW1 XA1E-BV302-R, U1 ABX00042

Commit message: save
Parts:
- added LED1, LED2, LED3, LED4, LED5: QTLP650C2TR, QTLP650C2TR:LEDC3216X130N, symbol QTLP650C2TR:QTLP650C2TR
- added R10: 1.5k. 1/2w, Resistor_SMD:R_1206_3216Metric_Pad1.30x1.75mm_HandSolder, symbol Device:R
- added R11: 200ohm, 1/10w, Resistor_SMD:R_1206_3216Metric_Pad1.30x1.75mm_HandSolder, symbol Device:R
- added R12, R7: 86ohm, 1/10w, Resistor_SMD:R_1206_3216Metric_Pad1.30x1.75mm_HandSolder, symbol Device:R
- added R13, R14, R8: 10k 1/8W, Resistor_SMD:R_1206_3216Metric_Pad1.30x1.75mm_HandSolder, symbol Device:R
- added R15: 1k 1/8w, Resistor_SMD:R_1206_3216Metric_Pad1.30x1.75mm_HandSolder, symbol Device:R
- DR1, DR2, DR3, DR4: Part Number (none) -> 3730
- IC1: Part Number (none) -> MC1413DR2G
- J1: value DRIVER 1 -> LED; Part Number (none) -> S4B-XH-SM4-TBLFSN
- J10, J11: Manufacturer_Part_Number FX30B-4S-3.81DSA -> (none); Part Number (none) -> FX30B-4S-3.81DSA
- J2: value DRIVER 3 -> LED; Part Number (none) -> S4B-XH-SM4-TBLFSN
- J3: value DRIVER 2 -> LED; Part Number (none) -> S4B-XH-SM4-TBLFSN
- J4: value DRIVER 4 -> LED; Part Number (none) -> S4B-XH-SM4-TBLFSN
- J5, J6, J7: Part Number (none) -> S4B-XH-SM4-TBLFSN
- Q1, Q2: Manufacturer_Part_Number BSS806NH6327XTSA1 -> (none); Part Number (none) -> BSS806NH6327XTSA1
- R1, R4, R6: value 10k -> 10k 1/8W; Part Number (none) -> RNCS1206BKE10K0
- R2: Part Number (none) -> RMCF1206FT4K02
- R3: value 1k -> 86ohm, 1/10w; Part Number (none) -> RC1206FR-0786R6L
- R5: value 1k -> 1k 1/8w; Part Number (none) -> RNCS1206BKE1K00
- SW1: Part Number (none) -> XA1E-BV302-R
- U1: Part Number (none) -> Portenta H7
- U2: Part Number (none) -> XB3-24AST-J
Connections:
- net 46_GPIO0_PC13 is gone; now on net GPIO6 GREEN LED: IC1.3 (IN_3)
- net 48_GPIO1_PC15 is gone; now on net GPIO5 YELLOW LED: IC1.2 (IN_2)
- net 50_GPIO2_PD4 is gone; now on net GPIO4 RED LED: IC1.1 (IN_1)
- net +24V: now also R10.2
- net +3.3V: now also U2.1 (VCC), R12.2
- net +5V: now also U1.J1_21 (VIN), U1.J1_41 (VIN), R11.2
- net 75_ANALOG_A1: now also R15.1; no longer R3.1
- net GND: now also J6.3, U1.J1_22 (GND), U1.J1_42 (GND), U1.J2_24 (GND_1), U1.J2_33 (GND_1), U1.J2_44 (GND_1), U1.J2_57 (GND_1), U1.J2_70 (GND_1), U2.10 (GND), LED1.1 (K), LED2.1 (K), LED3.1 (K), LED4.1 (K), LED5.1 (K), R15.2; no longer J6.2, R3.2
- net STEPPER_ENABLE: now also R7.2
- net ZIGBEE_IO: now also R3.2, U2.20 (AD0/DIO0)
- net D5 CLAMP: now reaches J6.4
- net D5 CLAMP: now also R1.2, U1.J2_61 (PWM_2)
- net at J5.2: now also R8.2; no longer IC1.16 (OUT_7)
- net at IC1.15 (OUT_6): now also R13.1; no longer J5.3
- net at J5.4: now also R14.2; no longer IC1.14 (OUT_5)
- net at J4.1: now also DR4.16 (AOUT1); no longer DR4.13 (BOUT2)
- net at J4.2: now also DR4.15 (AOUT2); no longer DR4.14 (BOUT1)
- net at J4.3: now also DR4.14 (BOUT1); no longer DR4.15 (AOUT2)
- net at J4.4: now also DR4.13 (BOUT2); no longer DR4.16 (AOUT1)
- net at J1.1: now also DR1.16 (AOUT1); no longer DR1.13 (BOUT2)
- net at J1.2: now also DR1.15 (AOUT2); no longer DR1.14 (BOUT1)
- net at J1.3: now also DR1.14 (BOUT1); no longer DR1.15 (AOUT2)
- net at J1.4: now also DR1.13 (BOUT2); no longer DR1.16 (AOUT1)
- net at J2.1: now also DR2.16 (AOUT1); no longer DR2.13 (BOUT2)
- net at J2.2: now also DR2.15 (AOUT2); no longer DR2.14 (BOUT1)
- net at J2.3: now also DR2.14 (BOUT1); no longer DR2.15 (AOUT2)
- net at J2.4: now also DR2.13 (BOUT2); no longer DR2.16 (AOUT1)
- net at DR3.13 (BOUT2): now also J3.4; no longer J3.1
- net at DR3.14 (BOUT1): now also J3.3; no longer J3.2
- net at DR3.15 (AOUT2): now also J3.2; no longer J3.3
- net at DR3.16 (AOUT1): now also J3.1; no longer J3.4
- net D4 STEP 4: now reaches DR4.4 (STEP/AIN1)
- net D4 STEP 4: now also U1.J2_63 (PWM_3)
- net GPIO3 DIR 4: now reaches DR4.5 (DIR/AIN2)
- net GPIO3 DIR 4: now also U1.J2_52 (GPIO_3)
- net at U1.J1_31 (GND), U1.J1_47 (GND), U1.J1_54 (GND): no longer U1.J1_22 (GND), U1.J1_42 (GND)
- net GPIO0 DIR 1: now reaches U1.J2_46 (GPIO_0)
- net GPIO0 DIR 1: now also DR1.5 (DIR/AIN2)
- net GPIO1 DIR 2: now reaches U1.J2_48 (GPIO_1)
- net GPIO1 DIR 2: now also DR2.5 (DIR/AIN2)
- net GPIO2 DIR 3: now reaches U1.J2_50 (GPIO_2)
- net GPIO2 DIR 3: now also DR3.5 (DIR/AIN2)
- net GPIO4 RED LED: now reaches U1.J2_54 (GPIO_4)
- net GPIO5 YELLOW LED: now reaches U1.J2_56 (GPIO_5)
- net GPIO6 GREEN LED: now reaches U1.J2_58 (GPIO_6)
- net D1 STEP 1: now reaches U1.J2_60 (PWM_6)
- net D1 STEP 1: now also DR1.4 (STEP/AIN1)
- net D3 STEP 3: now reaches U1.J2_65 (PWM_4)
- net D3 STEP 3: now also DR3.4 (STEP/AIN1)
- net D2 STEP 2: now reaches U1.J2_67 (PWM_5)
- net D2 STEP 2: now also DR2.4 (STEP/AIN1)
- net 52_GPIO3_PD5: no longer names the net of J6.1
- net 52_GPIO3_PD5: no longer R1.2
- net DO STEPPER ENABLE renamed D0 STEPPER ENABLE
- new net: J5.3, R13.2
- new net: LED1.2 (A), R3.1
- new net: LED4.2 (A), R11.1
- new net: LED2.2 (A), R7.1
- new net: LED5.2 (A), R12.1
- new net: IC1.14 (OUT_5), R14.1
- new net: LED3.2 (A), R10.1
- new net: IC1.16 (OUT_7), R8.1
- now unconnected: U1.J1_32 (VIN), U1.J1_48 (VIN), U1.J2_23 (VCC/+3V3), U1.J2_43 (VCC/+3V3), U1.J2_69 (VCC/+3V3)
Other:
- note added: "Error - (Fast Red Flashing) Idle - (Slow Pulse Yellow, 1) Running - (Slow Pulse Green) Estop - (Red Pulse, 1) internet / websocket comm down (flashing yellow, 2) zigbee comm down (Needs Help) initialization (All three on constant on start up, maybe count down) use count to distingush states"
- note added: "While the E-stop is connected this line is high, 3.3v This enables the gate on the estop line"
- moved on the sheet: J10, J11, Q1, R5, SW1, U2
