File: GR-LRR-POWER-PCB/GR-LRR-POWER-PCB.kicad_pcb (KiCad board)
At the start: 2 copper layers, 143.9 x 92.9 mm, 22 parts, among them IC1 TLV75533PDBVR, J1 BATT1, J2 BATT2, J3 POW_SW, J4 FX30B-4P-3.81DSA25, J5 FX30B-4P-3.81DSA25

Commit message: save
Routing:
- net BATT-: track 251.0 -> 250.5 mm
- net BATT+: track 278.3 -> 277.8 mm
Other:
- board text added: "GR-LRR-POWER-A1 12072023"
Changed lines of the file:
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@@
       (outputformat 1)
       (mirror false)
-      (drillshape 1)
+      (drillshape 0)
       (scaleselection 1)
-      (outputdirectory "")
+      (outputdirectory "GERBERS/")
     )
   )
@@
     (fp_line (start 2.25 1.6) (end 2.25 -1.6)
       (stroke (width 0.1) (type solid)) (layer "B.Fab"))
-    (pad "1" smd roundrect (at -2.1375 0 270) (size 1.575 3.4) (layers "B.Cu" "B.Paste" "B.Mask") (roundrect_rratio 0.15873)
+    (pad "1" smd roundrect (at -2.1375 0 270) (size 1.575 3.4) (layers "B.Cu" "B.Paste" "B.Mask") (roundrect_rratio 0.1587301587)
       (net 10 "BATT-") (pintype "passive"))
-    (pad "2" smd roundrect (at 2.1375 0 270) (size 1.575 3.4) (layers "B.Cu" "B.Paste" "B.Mask") (roundrect_rratio 0.15873)
+    (pad "2" smd roundrect (at 2.1375 0 270) (size 1.575 3.4) (layers "B.Cu" "B.Paste" "B.Mask") (roundrect_rratio 0.1587301587)
       (net 4 "GND") (pintype "passive"))
     (model "${KICAD6_3DMODEL_DIR}/Capacitor_SMD.3dshapes/C_1812_4532Metric.wrl"
@@
     (fp_line (start 1 0.625) (end 1 -0.625)
       (stroke (width 0.1) (type solid)) (layer "B.Fab"))
-    (pad "1" smd roundrect (at -1.0375 0 270) (size 1.175 1.45) (layers "B.Cu" "B.Paste" "B.Mask") (roundrect_rratio 0.212766)
+    (pad "1" smd roundrect (at -1.0375 0 270) (size 1.175 1.45) (layers "B.Cu" "B.Paste" "B.Mask") (roundrect_rratio 0.2127659574)
       (net 9 "BATT+") (pintype "passive"))
-    (pad "2" smd roundrect (at 1.0375 0 270) (size 1.175 1.45) (layers "B.Cu" "B.Paste" "B.Mask") (roundrect_rratio 0.212766)
+    (pad "2" smd roundrect (at 1.0375 0 270) (size 1.175 1.45) (layers "B.Cu" "B.Paste" "B.Mask") (roundrect_rratio 0.2127659574)
       (net 10 "BATT-") (pintype "passive"))
     (model "${KICAD6_3DMODEL_DIR}/Capacitor_SMD.3dshapes/C_0805_2012Metric.wrl"
@@
     (fp_line (start 2.25 1.6) (end 2.25 -1.6)
       (stroke (width 0.1) (type solid)) (layer "B.Fab"))
-    (pad "1" smd roundrect (at -2.1375 0 270) (size 1.575 3.4) (layers "B.Cu" "B.Paste" "B.Mask") (roundrect_rratio 0.15873)
+    (pad "1" smd roundrect (at -2.1375 0 270) (size 1.575 3.4) (layers "B.Cu" "B.Paste" "B.Mask") (roundrect_rratio 0.1587301587)
       (net 2 "+5V") (pintype "passive"))
-    (pad "2" smd roundrect (at 2.1375 0 270) (size 1.575 3.4) (layers "B.Cu" "B.Paste" "B.Mask") (roundrect_rratio 0.15873)
+    (pad "2" smd roundrect (at 2.1375 0 270) (size 1.575 3.4) (layers "B.Cu" "B.Paste" "B.Mask") (roundrect_rratio 0.1587301587)
       (net 5 "Net-(PS2-VIN)") (pintype "passive"))
     (model "${KICAD6_3DMODEL_DIR}/Capacitor_SMD.3dshapes/C_1812_4532Metric.wrl"
@@
     (fp_line (start 1 0.625) (end 1 -0.625)
       (stroke (width 0.1) (type solid)) (layer "B.Fab"))
-    (pad "1" smd roundrect (at -1.0375 0 270) (size 1.175 1.45) (layers "B.Cu" "B.Paste" "B.Mask") (roundrect_rratio 0.212766)
+    (pad "1" smd roundrect (at -1.0375 0 270) (size 1.175 1.45) (layers "B.Cu" "B.Paste" "B.Mask") (roundrect_rratio 0.2127659574)
       (net 2 "+5V") (pintype "passive"))
-    (pad "2" smd roundrect (at 1.0375 0 270) (size 1.175 1.45) (layers "B.Cu" "B.Paste" "B.Mask") (roundrect_rratio 0.212766)
+    (pad "2" smd roundrect (at 1.0375 0 270) (size 1.175 1.45) (layers "B.Cu" "B.Paste" "B.Mask") (roundrect_rratio 0.2127659574)
       (net 4 "GND") (pintype "passive"))
     (model "${KICAD6_3DMODEL_DIR}/Capacitor_SMD.3dshapes/C_0805_2012Metric.wrl"
@@
     (fp_line (start 3.65 2.15) (end -2.65 2.15)
       (stroke (width 0.1) (type solid)) (layer "B.Fab"))
-    (pad "1" smd roundrect (at -3.2 0 270) (size 2.25 2.55) (layers "B.Cu" "B.Paste" "B.Mask") (roundrect_rratio 0.111111)
+    (pad "1" smd roundrect (at -3.2 0 270) (size 2.25 2.55) (layers "B.Cu" "B.Paste" "B.Mask") (roundrect_rratio 0.1111111111)
       (net 2 "+5V") (pintype "passive"))
-    (pad "2" smd roundrect (at 3.2 0 270) (size 2.25 2.55) (layers "B.Cu" "B.Paste" "B.Mask") (roundrect_rratio 0.111111)
+    (pad "2" smd roundrect (at 3.2 0 270) (size 2.25 2.55) (layers "B.Cu" "B.Paste" "B.Mask") (roundrect_rratio 0.1111111111)
       (net 4 "GND") (pintype "passive"))
     (model "${KICAD6_3DMODEL_DIR}/Capacitor_Tantalum_SMD.3dshapes/CP_EIA-7343-15_Kemet-W.wrl"
@@
     (pad "MH4" thru_hole circle (at 48.3 -43.2) (size 4.8 4.8) (drill 3.2) (layers "*.Cu" "*.Mask")
       (net 19 "unconnected-(PS1-PadMH4)") (pinfunction "MH4") (pintype "passive"))
-    (model "${KIPRJMOD}/electronics_libraries/QSB30024S24/QSB30024S24.stp"
+    (model "QSB30024S24.stp"
       (offset (xyz 0 0 0))
       (scale (xyz 1 1 1))
@@
     (fp_line (start 1 0.625) (end 1 -0.625)
       (stroke (width 0.1) (type solid)) (layer "B.Fab"))
-    (pad "1" smd roundrect (at -1.0375 0 270) (size 1.175 1.45) (layers "B.Cu" "B.Paste" "B.Mask") (roundrect_rratio 0.212766)
+    (pad "1" smd roundrect (at -1.0375 0 270) (size 1.175 1.45) (layers "B.Cu" "B.Paste" "B.Mask") (roundrect_rratio 0.2127659574)
       (net 1 "+3.3V") (pintype "passive"))
-    (pad "2" smd roundrect (at 1.0375 0 270) (size 1.175 1.45) (layers "B.Cu" "B.Paste" "B.Mask") (roundrect_rratio 0.212766)
+    (pad "2" smd roundrect (at 1.0375 0 270) (size 1.175 1.45) (layers "B.Cu" "B.Paste" "B.Mask") (roundrect_rratio 0.2127659574)
       (net 4 "GND") (pintype "passive"))
     (model "${KICAD6_3DMODEL_DIR}/Capacitor_SMD.3dshapes/C_0805_2012Metric.wrl"
@@
   )
   (gr_text "BATT-" (at 41.798 101.136 90) (layer "F.SilkS")
+    (effects (font (size 1.5 1.5) (thickness 0.3) bold) (justify left bottom))
+  )
+  (gr_text "GR-LRR-POWER-A1\n12072023" (at 129.936 104.438) (layer "F.SilkS")
     (effects (font (size 1.5 1.5) (thickness 0.3) bold) (justify left bottom))
   )
@@
   (segment (start 37.684499 70.7885) (end 36.281999 69.386) (width 0.5) (layer "F.Cu") (net 9))
   (via (at 44.084 107.74) (size 0.8) (drill 0.4) (layers "F.Cu" "B.Cu") (net 9))
+  (segment (start 162.956 52.002) (end 162.956 99.104) (width 0.5) (layer "B.Cu") (net 9))
   (segment (start 44.846 69.386) (end 36.281999 69.386) (width 2) (layer "B.Cu") (net 9))
+  (segment (start 148.986 113.074) (end 49.418 113.074) (width 0.5) (layer "B.Cu") (net 9))
   (segment (start 56.8094 97.244323) (end 57.8508 98.285723) (width 2) (layer "B.Cu") (net 9))
-  (segment (start 163.21 52.256) (end 163.21 99.358) (width 0.5) (layer "B.Cu") (net 9))
+  (segment (start 157.526 46.572) (end 162.956 52.002) (width 0.5) (layer "B.Cu") (net 9))
   (segment (start 57.546 98.590523) (end 57.8508 98.285723) (width 2) (layer "B.Cu") (net 9))
   (segment (start 48.656 73.196) (end 44.846 69.386) (width 2) (layer "B.Cu") (net 9))
-  (segment (start 163.21 99.358) (end 149.494 113.074) (width 0.5) (layer "B.Cu") (net 9))
   (segment (start 48.656 97.244323) (end 48.656 73.196) (width 2) (layer "B.Cu") (net 9))
   (segment (start 49.418 113.074) (end 44.084 107.74) (width 0.5) (layer "B.Cu") (net 9))
-  (segment (start 157.526 46.572) (end 163.21 52.256) (width 0.5) (layer "B.Cu") (net 9))
   (segment (start 157.526 46.572) (end 154.526 46.572) (width 0.5) (layer "B.Cu") (net 9))
   (segment (start 57.546 102.074223) (end 57.546 98.590523) (width 2) (layer "B.Cu") (net 9))
-  (segment (start 149.494 113.074) (end 49.418 113.074) (width 0.5) (layer "B.Cu") (net 9))
   (segment (start 48.656 97.244323) (end 56.8094 97.244323) (width 2) (layer "B.Cu") (net 9))
-  (segment (start 162.448 99.13005) (end 149.26605 112.312) (width 0.5) (layer "B.Cu") (net 10))
+  (segment (start 162.956 99.104) (end 148.986 113.074) (width 0.5) (layer "B.Cu") (net 9))
+  (segment (start 49.858082 112.312) (end 39.444082 101.898) (width 0.5) (layer "B.Cu") (net 10))
   (segment (start 48.309677 101.898) (end 48.656 102.244323) (width 1) (layer "B.Cu") (net 10))
   (segment (start 36.556323 102.244323) (end 36.21 101.898) (width 2) (layer "B.Cu") (net 10))
-  (segment (start 162.448 55.304) (end 162.448 99.13005) (width 0.5) (layer "B.Cu") (net 10))
+  (segment (start 162.194 55.05) (end 162.194 98.85) (width 0.5) (layer "B.Cu") (net 10))
   (segment (start 65.583777 104.274223) (end 50.6859 104.274223) (width 2) (layer "B.Cu") (net 10))
-  (segment (start 157.526 50.382) (end 162.448 55.304) (width 0.5) (layer "B.Cu") (net 10))
-  (segment (start 49.858082 112.312) (end 39.444082 101.898) (width 0.5) (layer "B.Cu") (net 10))
+  (segment (start 157.526 50.382) (end 162.194 55.05) (width 0.5) (layer "B.Cu") (net 10))
   (segment (start 48.656 102.244323) (end 36.556323 102.244323) (width 2) (layer "B.Cu") (net 10))
   (segment (start 67.706 102.152) (end 65.583777 104.274223) (width 2) (layer "B.Cu") (net 10))
-  (segment (start 39.444082 101.898) (end 36.21 101.898) (width 0.5) (layer "B.Cu") (net 10))
+  (segment (start 162.194 98.85) (end 148.732 112.312) (width 0.5) (layer "B.Cu") (net 10))
+  (segment (start 148.732 112.312) (end 49.858082 112.312) (width 0.5) (layer "B.Cu") (net 10))
   (segment (start 157.526 50.382) (end 154.526 50.382) (width 0.5) (layer "B.Cu") (net 10))
   (segment (start 67.706 102.152) (end 88.788 102.152) (width 2) (layer "B.Cu") (net 10))
-  (segment (start 149.26605 112.312) (end 49.858082 112.312) (width 0.5) (layer "B.Cu") (net 10))
+  (segment (start 39.444082 101.898) (end 36.21 101.898) (width 0.5) (layer "B.Cu") (net 10))
   (segment (start 88.788 102.152) (end 89.804 101.136) (width 2) (layer "B.Cu") (net 10))
   (segment (start 89.296 102.152) (end 89.804 101.644) (width 2) (layer "B.Cu") (net 10))
