File: GR-LRR-POWER-PCB/GR-LRR-POWER-PCB.kicad_sch (KiCad schematic)
At the start: 26 parts, among them IC1 TLV75533PDBVR, J3 BATT1, J4 BATT2, J4 FX30B-4P-3.81DSA25, J4 POW_SW, J5 FX30B-4P-3.81DSA25

Commit message: save
Parts:
- C1, C2, C3: Part Number (none) -> 100PX220MEFC12.5X20
- D1: Part Number (none) -> SMCJ40A
- IC1: Manufacturer_Part_Number TLV75533PDBVR -> (none); Part Number (none) -> TLV75533PDBVR
- J3, J4: Part Number (none) -> 2604-1102
- J4, J5: Manufacturer_Part_Number FX30B-4P-3.81DSA25 -> (none); Part Number (none) -> FX30B-4P-3.81DSA25
- L1: Manufacturer_Part_Number 047700 -> (none); Part Number (none) -> 047700
- PS1: Manufacturer_Part_Number QSB30024S24 -> (none); Part Number (none) -> QSB30024S24
- PS2: Part Number (none) -> PYBE20-Q24-S5
