File: GR-LRR-CONTROL/GR-LRR-CONTROL.kicad_pcb (KiCad board)
At the start: 2 copper layers, 213.7 x 137.6 mm, 110 parts, among them IC1 TJA1049T,118, IC2 MC1413DR2G, J1 87833-1019, J10 430451000, J11 87833-1019, J12 10018783-10101TLF, J13 430450200, J14 430451000, J15 87833-1019, J16 10018783-10101TLF, J17 430450200, J18 691137710002, J19 901362104, J2 430451000, J20 901362102, J21 ENC1, J22 ENC2, J23 901362104, J24 LED, J25 UT1, J26 UT2, J27 901362103, J28 901362103, J29 901362103, J3 10018783-10101TLF, J30 901362103, J31 901362103, J32 Conn_02x07_Odd_Even, J33 Conn_01x03, J34 Conn_01x03, J35 THD-20-R, J36 USB_OTG, J37 690-008-221-904, J38 690-008-221-904, J4 430450200, J5 DT13-08PB, J6 430451000, J7 87833-1019, J8 10018783-10101TLF, J9 430450200, Q1 BSS806NH6327XTSA1, Q2 BSS806NH6327XTSA1, U1 ABX00042, U10 USB2514B-I/M2, U11 TPD4EUSB30, U12 AP22653W6, U2 INA260AIPWR, U3 1k, U5 YC248-JR-0710KL, U6 PCA9685PW, U7 74LVC1G07SE-7, U8 74LVC1G07SE-7, U9 FSUSB42MUX, Y1 24MHz

Commit message: purchasing A3 power
Parts:
- removed J13, J17, J4, J9: 430450200, avid_footprints:430450200
- removed J35: THD-20-R, Connector_PinHeader_2.54mm:PinHeader_2x20_P2.54mm_Vertical
- removed Q2: BSS806NH6327XTSA1, avid_footprints:SOT95P240X110-3N
- added J39: Conn_02x12_Counter_Clockwise, Connector_PinHeader_2.54mm:PinHeader_2x12_P2.54mm_Vertical, F.Cu at (159.6, 132.0)
- added R31: 120, Resistor_SMD:R_1206_3216Metric_Pad1.30x1.75mm_HandSolder, F.Cu at (150.4, 169.9)
- U1: footprint avid_footprints:MODULE_ABX00042 -> avid_footprints:MODULE_ABX00042_2
- moved J32 425.5 mm to (235.0, 155.5), turned to 180 degrees
- moved R22 412.8 mm to (239.2, 118.9), turned to 90 degrees
- moved J34 412.1 mm to (232.6, 104.2)
- moved R20 408.2 mm to (236.2, 114.0), turned to -90 degrees
- moved R21 407.4 mm to (232.6, 114.0), turned to -90 degrees
- moved TP2 404.7 mm to (240.2, 121.4), turned to -90 degrees
- moved U8 404.5 mm to (240.2, 116.2), turned to -90 degrees
- moved R19 402.3 mm to (240.1, 134.8), turned to -90 degrees
- moved D2 402.2 mm to (239.5, 124.5), turned to -90 degrees
- moved J33 400.9 mm to (232.6, 123.9), turned to 180 degrees
- moved D1 398.0 mm to (239.8, 129.0), turned to 90 degrees
- moved TP1 394.7 mm to (239.0, 132.2), turned to 90 degrees
- moved U7 384.2 mm to (232.2, 135.2), turned to 180 degrees
- moved R3 263.5 mm to (102.4, 97.4)
- moved R1 211.4 mm to (158.9, 138.6), turned to 0 degrees
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Connections:
- net DVR_CAN_Hi_1 renamed DVR_CAN_1_+
- net DVR_CAN_Lo_1 renamed DVR_CAN_1_-
- J12 pad A21: DVR_+Vmot_3 -> 18V
- J12 pad A22: DVR_+Vmot_3 -> 18V
- J12 pad B21: DVR_+Vmot_3 -> 18V
- J12 pad B22: DVR_+Vmot_3 -> 18V
- J16 pad A21: DVR_+Vmot_4 -> 18V
- J16 pad A22: DVR_+Vmot_4 -> 18V
- J16 pad B21: DVR_+Vmot_4 -> 18V
- J16 pad B22: DVR_+Vmot_4 -> 18V
- J18 pad 2: STEPPER_ENABLE -> D0 ESTOP DETECT
- J3 pad A21: DVR_+Vmot_1 -> 18V
- J3 pad A22: DVR_+Vmot_1 -> 18V
- J3 pad B21: DVR_+Vmot_1 -> 18V
- J3 pad B22: DVR_+Vmot_1 -> 18V
- J8 pad A21: DVR_+Vmot_2 -> 18V
- J8 pad A22: DVR_+Vmot_2 -> 18V
- J8 pad B21: DVR_+Vmot_2 -> 18V
- J8 pad B22: DVR_+Vmot_2 -> 18V
- Q1 pad 1: D0 STEPPER ENABLE -> ZIGBEE_IO
- Q1 pad 3: Net-(Q1-D) -> 3.3V
- R13 pad 2: STEPPER_ENABLE -> D0 ESTOP DETECT
- R14 pad 1: STEPPER_ENABLE -> D0 ESTOP DETECT
- U1 pad J1_32: unconnected-(U1A-VIN-PadJ1_32) -> 5V
- U1 pad J1_48: unconnected-(U1A-VIN-PadJ1_48) -> 5V
- U1 pad J2_46: GPIO0 DIR 1 -> GPIO0
- U1 pad J2_48: GPIO1 DIR 2 -> GPIO1
- U1 pad J2_50: GPIO2 DIR 3 -> GPIO2
- U1 pad J2_52: GPIO3 DIR 4 -> GPIO3
- U1 pad J2_59: unconnected-(U1B-PWM_1-PadJ2_59) -> D6
- U1 pad J2_60: D1 STEP 1 -> D1
- U1 pad J2_61: CLAMP_C -> D5 Clamp
- U1 pad J2_62: D0 STEPPER ENABLE -> D0 ESTOP DETECT
- U1 pad J2_63: D4 STEP 4 -> D4
- U1 pad J2_65: D3 STEP 3 -> D3
- U1 pad J2_67: D2 STEP 2 -> D2
- U1 pad J2_74: unconnected-(U1B-ADC_A4-PadJ2_74) -> A4
- U1 pad J2_76: unconnected-(U1B-ADC_A5-PadJ2_76) -> A5
- U1 pad J2_78: unconnected-(U1B-ADC_A6-PadJ2_78) -> A6
- U1 pad J2_79: unconnected-(U1B-ADC_A3-PadJ2_79) -> A3
- U1 pad J2_80: unconnected-(U1B-ADC_A7-PadJ2_80) -> A7
Routing:
- net H7_I2C0_SCL: track 0.00 -> 225.1 mm, vias 0 -> 3
- net H7_I2C0_SDA: track 0.00 -> 211.7 mm, vias 0 -> 2
- net 24V: track 0.00 -> 163.8 mm
- net GND: track 0.00 -> 151.0 mm, vias 0 -> 54
- net 18V: track 0.00 -> 146.7 mm
- net D0 ESTOP DETECT: track 0.00 -> 136.5 mm, vias 0 -> 1
- net DVR_CAN_1_-: track 0.00 -> 125.4 mm, vias 0 -> 2
- net UT2_77_A2: track 0.00 -> 106.6 mm, vias 0 -> 2
- net DVR_+5VOUT_2: track 0.00 -> 100.6 mm
- net DVR_+5VOUT_3: track 0.00 -> 98.4 mm
- net BAT_MON_73_A0: track 0.00 -> 96.2 mm, vias 0 -> 2
- net DVR_C/B+_3: track 0.00 -> 95.6 mm
- net UT1_75_A1: track 0.00 -> 95.0 mm, vias 0 -> 2
- net ENCODER2_PHASEZ: track 0.00 -> 93.8 mm
- net DVR_+5VOUT_1: track 0.00 -> 93.5 mm
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- added copper zone on F.Cu, net 18V
- added copper zone on F.Cu, net 18V_IN
- added copper zone on In1.Cu, net 3.3V
- added copper zone on In2.Cu, net 5V
- added copper zone on B.Cu, net GND
- added copper zone on F.Cu, net GND
Other:
- copper layers 2 -> 4
