File: GR-LRR-CONTROL/CM4_GPIO.kicad_sch (KiCad schematic)
At the start: 15 parts, among them J11 Conn_02x07_Odd_Even, J12 Conn_01x03, J13 Conn_01x03, J14 THD-20-R, U11 74LVC1G07SE-7, U12 74LVC1G07SE-7

Commit message: purchasing A3 power
Parts:
- removed J14: THD-20-R, Connector_PinHeader_2.54mm:PinHeader_2x20_P2.54mm_Vertical, symbol Connector_Generic:Conn_02x20_Odd_Even
Changed lines of the file:
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@@
 	)
 	(junction
-		(at 152.4 41.91)
-		(diameter 1.016)
-		(color 0 0 0 0)
-	)
-	(junction
 		(at 100.076 118.11)
 		(diameter 1.016)
@@
 	(wire
 		(pts
-			(xy 140.97 41.91) (xy 152.4 41.91)
-		)
-		(stroke
-			(width 0)
-			(type solid)
-		)
-	)
-	(wire
-		(pts
 			(xy 161.798 145.542) (xy 175.768 145.542)
 		)
@@
 	(wire
 		(pts
-			(xy 154.94 41.91) (xy 152.4 41.91)
+			(xy 140.97 41.91) (xy 154.94 41.91)
 		)
 		(stroke
@@
 					(unit 1)
 				)
-			)
-		)
-	)
-	(symbol
-		(lib_id "Connector_Generic:Conn_02x20_Odd_Even")
-		(at 157.48 46.99 0)
-		(unit 1)
-		(exclude_from_sim no)
-		(in_bom yes)
-		(on_board yes)
-		(dnp no)
-		(property "Reference" "J14"
-			(at 166.37 21.59 0)
-			(effects
-				(font
-					(size 1.27 1.27)
-				)
-			)
-		)
-		(property "Value" "THD-20-R"
-			(at 158.75 20.9296 0)
-			(effects
-				(font
-					(size 1.27 1.27)
-				)
-			)
-		)
-		(property "Footprint" "Connector_PinHeader_2.54mm:PinHeader_2x20_P2.54mm_Vertical"
-			(at 157.48 46.99 0)
-			(effects
-				(font
-					(size 1.27 1.27)
-				)
-				(hide yes)
-			)
-		)
-		(property "Datasheet" "https://www.toby.co.uk/uploads/publications/1673.pdf"
-			(at 157.48 46.99 0)
-			(effects
-				(font
-					(size 1.27 1.27)
-				)
-				(hide yes)
-			)
-		)
-		(property "Description" ""
-			(at 157.48 46.99 0)
-			(effects
-				(font
-					(size 1.27 1.27)
-				)
-				(hide yes)
-			)
-		)
-		(property "Field4" "Toby"
-			(at 157.48 46.99 0)
-			(effects
-				(font
-					(size 1.27 1.27)
-				)
-				(hide yes)
-			)
-		)
-		(property "Field5" "THD-20-R"
-			(at 157.48 46.99 0)
-			(effects
-				(font
-					(size 1.27 1.27)
-				)
-				(hide yes)
-			)
-		)
-		(property "Field6" "THD-20-R"
-			(at 157.48 46.99 0)
-			(effects
-				(font
-					(size 1.27 1.27)
-				)
-				(hide yes)
-			)
-		)
-		(property "Field7" "Toby"
-			(at 157.48 46.99 0)
-			(effects
-				(font
-					(size 1.27 1.27)
-				)
-				(hide yes)
-			)
-		)
-		(property "Field8" "UCON00511"
-			(at 157.48 46.99 0)
-			(effects
-				(font
-					(size 1.27 1.27)
-				)
-				(hide yes)
-			)
-		)
-		(property "Part Description" "PinHeader_2x20_P2.54mm_Vertical"
-			(at 157.48 46.99 0)
-			(effects
-				(font
-					(size 1.27 1.27)
-				)
-				(hide yes)
-			)
-		)
-		(pin "1"
-		)
-		(pin "10"
-		)
-		(pin "11"
-		)
-		(pin "12"
-		)
-		(pin "13"
-		)
-		(pin "14"
-		)
-		(pin "15"
-		)
-		(pin "16"
-		)
-		(pin "17"
-		)
-		(pin "18"
-		)
-		(pin "19"
-		)
-		(pin "2"
-		)
-		(pin "20"
-		)
-		(pin "21"
-		)
-		(pin "22"
-		)
-		(pin "23"
-		)
-		(pin "24"
-		)
-		(pin "25"
-		)
-		(pin "26"
-		)
-		(pin "27"
-		)
-		(pin "28"
-		)
-		(pin "29"
-		)
-		(pin "3"
-		)
-		(pin "30"
-		)
-		(pin "31"
-		)
-		(pin "32"
-		)
-		(pin "33"
-		)
-		(pin "34"
-		)
-		(pin "35"
-		)
-		(pin "36"
-		)
-		(pin "37"
-		)
-		(pin "38"
-		)
-		(pin "39"
-		)
-		(pin "4"
-		)
-		(pin "40"
-		)
-		(pin "5"
-		)
-		(pin "6"
-		)
-		(pin "7"
-		)
-		(pin "8"
-		)
-		(pin "9"
-		)
-		(instances
-			(project "GR-LRR-CONTROL-PCB"
-				(path "/3c88e67a-9fbd-4775-aa51-31d4ca1ce189/47ad118d-a453-435b-a9d8-083c942d52a2"
-					(reference "J14")
-					(unit 1)
-				)
-			)
-			(project "GR-LRR-CONTROL"
-				(path "/7e750e3c-c787-4adb-8081-69356fc148e5/b7f2159b-e50e-4dd7-8990-15596336c7e2"
-					(reference "J35")
-					(unit 1)
-				)

Commit message: finished routing
Parts:
- added J4: Conn_02x12_Counter_Clockwise, Connector_PinHeader_2.54mm:PinHeader_2x12_P2.54mm_Vertical, symbol Connector_Generic:Conn_02x12_Counter_Clockwise
Connections:
- net +3.3v: now also J4.1 (Pin_1), J4.9 (Pin_9)
- net +5v: now also J4.23 (Pin_23), J4.24 (Pin_24)
- net GND: now also J4.15 (Pin_15), J4.18 (Pin_18), J4.22 (Pin_22), J4.5 (Pin_5)
- net GPIO10: now also J4.10 (Pin_10)
- net GPIO11: now also J4.12 (Pin_12)
- net GPIO17: now also J4.6 (Pin_6)
- net GPIO18: now also J4.19 (Pin_19)
- net GPIO2: now also J4.2 (Pin_2)
- net GPIO22: now also J4.8 (Pin_8)
- net GPIO23: now also J4.17 (Pin_17)
- net GPIO24: now also J4.16 (Pin_16)
- net GPIO25: now also J4.14 (Pin_14)
- net GPIO27: now also J4.7 (Pin_7)
- net GPIO3: now also J4.3 (Pin_3)
- net GPIO4: now also J4.4 (Pin_4)
- net GPIO8: now also J4.13 (Pin_13)
- net GPIO9: now also J4.11 (Pin_11)
- net RPI_GPIO_14_TX: now also J4.21 (Pin_21)
- net RPI_GPIO_15_RX: now also J4.20 (Pin_20)
Other:
- note added: "1. 3.3V 3. GPIO3 5. GND 7. GPIO27 9. 3.3V 11. GPIO9 13. GPIO8 15. GND 17. GPIO23 19. GPIO18 21. GPIO14 23. 5V"
- note added: "2. G2 4. G4 6. G17 8. G22 10. G10 12. G11 14. G25 16. G24 18. GND 20. G15 22. GND 24. 5V"
Changed lines of the file:
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@@
 	(wire
 		(pts
-			(xy 140.97 41.91) (xy 154.94 41.91)
+			(xy 140.97 41.91) (xy 152.4 41.91)
 		)
 		(stroke
@@
 		)
 	)
+	(text "1. 3.3V\n3. GPIO3\n5. GND\n7. GPIO27\n9. 3.3V\n11. GPIO9\n13. GPIO8\n15. GND\n17. GPIO23\n19. GPIO18\n21. GPIO14\n23. 5V"
+		(exclude_from_sim no)
+		(at 181.61 50.292 0)
+		(effects
+			(font
+				(size 1.27 1.27)
+			)
+			(justify left)
+		)
+	)
 	(text "Activity LED"
 		(exclude_from_sim no)
@@
 		)
 	)
+	(text "2. G2\n4. G4\n6. G17\n8. G22\n10. G10\n12. G11\n14. G25\n16. G24\n18. GND\n20. G15\n22. GND\n24. 5V"
+		(exclude_from_sim no)
+		(at 212.09 51.054 0)
+		(effects
+			(font
+				(size 1.27 1.27)
+			)
+		)
+	)
 	(text "A button between pins 13-14 can be used to wake up compute module from power down\n\n"
 		(exclude_from_sim no)
@@
 					(unit 1)
 				)
+			)
+		)
+	)
+	(symbol
+		(lib_id "Connector_Generic:Conn_02x12_Counter_Clockwise")
+		(at 157.48 36.83 0)
+		(unit 1)
+		(exclude_from_sim no)
+		(in_bom yes)
+		(on_board yes)
+		(dnp no)
+		(fields_autoplaced yes)
+		(property "Reference" "J4"
+			(at 158.75 17.78 0)
+			(effects
+				(font
+					(size 1.27 1.27)
+				)
+			)
+		)
+		(property "Value" "Conn_02x12_Counter_Clockwise"
+			(at 158.75 20.32 0)
+			(effects
+				(font
+					(size 1.27 1.27)
+				)
+			)
+		)
+		(property "Footprint" "Connector_PinHeader_2.54mm:PinHeader_2x12_P2.54mm_Vertical"
+			(at 157.48 36.83 0)
+			(effects
+				(font
+					(size 1.27 1.27)
+				)
+				(hide yes)
+			)
+		)
+		(property "Datasheet" "~"
+			(at 157.48 36.83 0)
+			(effects
+				(font
+					(size 1.27 1.27)
+				)
+				(hide yes)
+			)
+		)
+		(property "Description" "Generic connector, double row, 02x12, counter clockwise pin numbering scheme (similar to DIP package numbering), script generated (kicad-library-utils/schlib/autogen/connector/)"
+			(at 157.48 36.83 0)
+			(effects
+				(font
+					(size 1.27 1.27)
+				)
+				(hide yes)
+			)
+		)
+		(pin "17"
+		)
+		(pin "1"
+		)
+		(pin "12"
+		)
+		(pin "2"
+		)
+		(pin "20"
+		)
+		(pin "8"
+		)
+		(pin "11"
+		)
+		(pin "10"
+		)
+		(pin "16"
+		)
+		(pin "4"
+		)
+		(pin "22"
+		)
+		(pin "6"
+		)
+		(pin "14"
+		)
+		(pin "9"
+		)
+		(pin "7"
+		)
+		(pin "24"
+		)
+		(pin "3"
+		)
+		(pin "13"
+		)
+		(pin "23"
+		)
+		(pin "21"
+		)
+		(pin "15"
+		)
+		(pin "18"
+		)
+		(pin "19"
+		)
+		(pin "5"
+		)
+		(instances
+			(project "GR-LRR-CONTROL"
+				(path "/7e750e3c-c787-4adb-8081-69356fc148e5/b7f2159b-e50e-4dd7-8990-15596336c7e2"
+					(reference "J4")
+					(unit 1)
+				)

Commit message: ordered power and control A4
Parts:
- added CR2: PMEG6020ER_115, avid_footprints:CFP3_SOD123W_NEX, symbol avid_symbols:PMEG6020ER_115
Connections:
- net +5v: now also CR2.2; no longer Module1.77 (+5v_(Input)), Module1.79 (+5v_(Input)), Module1.81 (+5v_(Input)), Module1.83 (+5v_(Input)), Module1.85 (+5v_(Input)), Module1.87 (+5v_(Input))
- new net: CR2.1, Module1.77 (+5v_(Input)), Module1.79 (+5v_(Input)), Module1.81 (+5v_(Input)), Module1.83 (+5v_(Input)), Module1.85 (+5v_(Input)), Module1.87 (+5v_(Input))
Changed lines of the file:
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@@
 	(wire
 		(pts
+			(xy 130.81 115.57) (xy 124.46 115.57)
+		)
+		(stroke
+			(width 0)
+			(type default)
+		)
+	)
+	(wire
+		(pts
 			(xy 140.97 49.53) (xy 152.4 49.53)
 		)
@@
 	(wire
 		(pts
-			(xy 100.076 115.57) (xy 114.046 115.57)
+			(xy 100.076 115.57) (xy 114.3 115.57)
 		)
 		(stroke
@@
 		)
 	)
+	(label "+5v"
+		(at 128.27 115.57 180)
+		(fields_autoplaced yes)
+		(effects
+			(font
+				(size 1.27 1.27)
+			)
+			(justify right bottom)
+		)
+	)
 	(label "SYNC_IN"
 		(at 87.63 172.72 180)
@@
 		)
 	)
-	(label "+5v"
-		(at 106.426 115.57 180)
-		(fields_autoplaced yes)
-		(effects
-			(font
-				(size 1.27 1.27)
-			)
-			(justify right bottom)
-		)
-	)
 	(label "SYNC_OUT"
 		(at 33.02 39.37 180)
@@
 		)
 	)
-	(hierarchical_label "+5v"
-		(shape input)
-		(at 114.046 115.57 0)
-		(fields_autoplaced yes)
-		(effects
-			(font
-				(size 1.27 1.27)
-			)
-			(justify left)
-		)
-	)
 	(hierarchical_label "GLOBAL_EN"
 		(shape input)
@@
 		)
 	)
+	(hierarchical_label "+5v"
+		(shape input)
+		(at 130.81 115.57 0)
+		(fields_autoplaced yes)
+		(effects
+			(font
+				(size 1.27 1.27)
+			)
+			(justify left)
+		)
+	)
 	(hierarchical_label "SCL0"
 		(shape output)
@@
 					(unit 1)
 				)
+			)
+		)
+	)
+	(symbol
+		(lib_id "avid_symbols:PMEG6020ER_115")
+		(at 124.46 115.57 180)
+		(unit 1)
+		(exclude_from_sim no)
+		(in_bom yes)
+		(on_board yes)
+		(dnp no)
+		(fields_autoplaced yes)
+		(property "Reference" "CR2"
+			(at 119.38 109.22 0)
+			(effects
+				(font
+					(size 1.524 1.524)
+				)
+			)
+		)
+		(property "Value" "PMEG6020ER_115"
+			(at 119.38 111.76 0)
+			(effects
+				(font
+					(size 1.524 1.524)
+				)
+			)
+		)
+		(property "Footprint" "avid_footprints:CFP3_SOD123W_NEX"
+			(at 124.46 115.57 0)
+			(effects
+				(font
+					(size 1.27 1.27)
+					(italic yes)
+				)
+				(hide yes)
+			)
+		)
+		(property "Datasheet" "PMEG6020ER_115"
+			(at 124.46 115.57 0)
+			(effects
+				(font
+					(size 1.27 1.27)
+					(italic yes)
+				)
+				(hide yes)
+			)
+		)
+		(property "Description" ""
+			(at 124.46 115.57 0)
+			(effects
+				(font
+					(size 1.27 1.27)
+				)
+				(hide yes)
+			)
+		)
+		(pin "1"
+		)
+		(pin "2"
+		)
+		(instances
+			(project "GR-LRR-CONTROL"
+				(path "/7e750e3c-c787-4adb-8081-69356fc148e5/b7f2159b-e50e-4dd7-8990-15596336c7e2"
+					(reference "CR2")
+					(unit 1)
+				)

Commit message: upload
Parts:
- CR2: Part Number (none) -> PMEG6020ER_115
- D1: Field5 LTST-S270KGKT -> (none); Part Number (none) -> LTST-S270KGKT
- D2: Field5 LTST-S270KRKT -> (none); Part Number (none) -> LTST-S270KRKT
- Module1: Part Number (none) -> SC0675
- R49, R52: Field6 RK73H1ETTP1001F -> (none); Part Number (none) -> RK73H1ETTP1001F
- U11, U12: Part Number (none) -> 74LVC1G07SE-7
Changed lines of the file:
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@@
+			)
+		)
+		(property "Part Number" "74LVC1G07SE-7"
+			(at 183.388 145.542 0)
+			(effects
+				(font
+					(size 1.27 1.27)
+				)
+				(hide yes)
 			)
 		)
@@
 			)
 		)
+		(property "Part Number" "74LVC1G07SE-7"
+			(at 27.94 180.34 0)
+			(effects
+				(font
+					(size 1.27 1.27)
+				)
+				(hide yes)
+			)
+		)
 		(pin "2"
 		)
@@
 			)
 		)
+		(property "Part Number" "SC0675"
+			(at 72.136 74.93 0)
+			(effects
+				(font
+					(size 1.27 1.27)
+				)
+				(hide yes)
+			)
+		)
 		(pin "1"
 		)
@@
 			)
 		)
-		(property "Field5" "LTST-S270KGKT"
+		(property "Part Number" "LTST-S270KGKT"
 			(at 116.84 25.4 0)
 			(effects
@@
 			)
 		)
-		(property "Field6" "RK73H1ETTP1001F"
+		(property "Part Number" "RK73H1ETTP1001F"
 			(at 116.84 38.1 0)
 			(effects
@@
 			)
 		)
-		(property "Field5" "	LTST-S270KRKT"
+		(property "Part Number" "	LTST-S270KRKT"
 			(at 191.008 126.492 0)
 			(effects
@@
 			)
 		)
-		(property "Field6" "RK73H1ETTP1001F"
+		(property "Part Number" "RK73H1ETTP1001F"
 			(at 191.008 135.382 0)
 			(effects
@@
 			(at 124.46 115.57 0)
 			(effects
+				(font
+					(size 1.27 1.27)
+				)
+				(hide yes)
+			)
+		)
+		(property "Part Number" "PMEG6020ER_115"
+			(at 124.46 115.57 0)
+			(effects
