File: GR-LRR-CONTROL/CM4_HighSpeed.kicad_sch (KiCad schematic)
At the start: 1 part

Commit message: finished routing
Connections:
- net USB2_N renamed USB2_-
- net USB2_P renamed USB2_+
Changed lines of the file:
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@@
 		)
 	)
-	(hierarchical_label "USB2_P"
+	(hierarchical_label "USB2_+"
 		(shape bidirectional)
 		(at 109.22 31.75 0)
@@
 		)
 	)
-	(hierarchical_label "USB2_N"
+	(hierarchical_label "USB2_-"
 		(shape bidirectional)
 		(at 109.22 29.21 0)

Commit message: upload
Parts:
- Module1: Part Number (none) -> SC0675
Changed lines of the file:
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@@
+			)
+		)
+		(property "Part Number" "SC0675"
+			(at -67.31 87.63 0)
+			(effects
+				(font
+					(size 1.27 1.27)
+				)
+				(hide yes)
 			)
 		)
