File: GR-LRR-CONTROL/GR-LRR-CONTROL.kicad_sch (KiCad schematic)
At the start: 64 parts, among them IC1 TJA1049T,118, IC2 MC1413DR2G, J1 87833-1019, J10 430451000, J11 87833-1019, J12 10018783-10101TLF, J13 430450200, J14 430451000, J15 87833-1019, J16 10018783-10101TLF, J17 430450200, J18 691137710002, J19 901362104, J2 430451000, J20 901362102, J21 ENC1, J22 ENC2, J23 901362104, J24 LED, J25 UT1, J26 UT2, J27 901362103, J28 901362103, J29 901362103, J3 10018783-10101TLF, J30 901362103, J31 901362103, J4 430450200, J5 DT13-08PB, J6 430451000, J7 87833-1019, J8 10018783-10101TLF, J9 430450200, Q1 BSS806NH6327XTSA1, Q2 BSS806NH6327XTSA1, SW1 XA1E-BV302-R, U1 ABX00042, U2 INA260AIPWR, U3 1k, U5 YC248-JR-0710KL, U6 PCA9685PW

Commit message: purchasing A3 power
Parts:
- removed J13, J17, J4, J9: 430450200, avid_footprints:430450200, symbol avid_symbols:430450200
- removed Q2: BSS806NH6327XTSA1, SOT95P240X110-3N, symbol BSS806NH6327XTSA1:BSS806NH6327XTSA1
- added J39: Conn_02x12_Counter_Clockwise, Connector_PinHeader_2.54mm:PinHeader_2x12_P2.54mm_Vertical, symbol Connector_Generic:Conn_02x12_Counter_Clockwise
- added R31: 120, Resistor_SMD:R_1206_3216Metric_Pad1.30x1.75mm_HandSolder, symbol Device:R
- U1: footprint avid_footprints:MODULE_ABX00042 -> avid_footprints:MODULE_ABX00042_2
Connections:
- net 18V_IN is gone; now on net BATT+: J5.3, J5.4, U2.1 (IN+), U2.12 (VBUS), U2.2 (IN+), U2.3 (IN+)
- net DVR_+Vmot_1 is gone; now on net 18V: J3.A21, J3.A22, J3.B21, J3.B22
- net DVR_+Vmot_2 is gone; now on net 18V: J8.A21, J8.A22, J8.B21, J8.B22
- net DVR_+Vmot_3 is gone; now on net 18V: J12.A21, J12.A22, J12.B21, J12.B22
- net DVR_+Vmot_4 is gone; now on net 18V: J16.A21, J16.A22, J16.B21, J16.B22
- net STEPPER_ENABLE is gone; now on net D0 ESTOP DETECT: J18.2, R13.2, R14.1
- net 3.3V: now also Q1.3 (D)
- net 5V: now also U1.J1_32 (VIN), U1.J1_48 (VIN)
- net BAT_MON_73_A0: now also J39.17 (Pin_17)
- net CLAMP_C: no longer U1.J2_61 (PWM_2)
- net D10 CIPO: now also J39.7 (Pin_7)
- net D7 CS: now also J39.9 (Pin_9)
- net D8 COPI: now also J39.6 (Pin_6)
- net D9 CK: now also J39.8 (Pin_8)
- net GPIO4 RED LED: now also J39.1 (Pin_1)
- net UT1_75_A1: now also J39.18 (Pin_18)
- net UT2_77_A2: now also J39.19 (Pin_19)
- net ZIGBEE_IO: now also Q1.1 (G)
- net D6: now reaches U1.J2_59 (PWM_1)
- net D6: now also J39.16 (Pin_16)
- net A4: now reaches U1.J2_74 (ADC_A4)
- net A4: now also J39.21 (Pin_21)
- net A5: now reaches U1.J2_76 (ADC_A5)
- net A5: now also J39.22 (Pin_22)
- net A6: now reaches U1.J2_78 (ADC_A6)
- net A6: now also J39.23 (Pin_23)
- net A3: now reaches U1.J2_79 (ADC_A3)
- net A3: now also J39.20 (Pin_20)
- net A7: now reaches U1.J2_80 (ADC_A7)
- net A7: now also J39.24 (Pin_24)
- net D0 STEPPER ENABLE renamed D0 ESTOP DETECT
- net D0 ESTOP DETECT: now also J39.10 (Pin_10); no longer Q1.1 (G)
- net D1 STEP 1 renamed D1
- net D1: now also J39.11 (Pin_11)
- net D2 STEP 2 renamed D2
- net D2: now also J39.12 (Pin_12)
- net D3 STEP 3 renamed D3
- net D3: now also J39.13 (Pin_13)
- net D4 STEP 4 renamed D4
- net D4: now also J39.14 (Pin_14)
- net DVR_CAN_Hi_1 renamed DVR_CAN_1_+
- net DVR_CAN_1_+: now also R31.1
- net DVR_CAN_Lo_1 renamed DVR_CAN_1_-
- net DVR_CAN_1_-: now also R31.2
- net GPIO0 DIR 1 renamed GPIO0
- net GPIO0: now also J39.5 (Pin_5)
- net GPIO1 DIR 2 renamed GPIO1
- net GPIO1: now also J39.4 (Pin_4)
- net GPIO2 DIR 3 renamed GPIO2
- net GPIO2: now also J39.3 (Pin_3)
- net GPIO3 DIR 4 renamed GPIO3
- net GPIO3: now also J39.2 (Pin_2)
- new net D5 Clamp: J39.15 (Pin_15), U1.J2_61 (PWM_2)

Commit message: finished routing
Parts:
- removed C1: 0.1uF, Capacitor_SMD:C_1206_3216Metric_Pad1.33x1.80mm_HandSolder, symbol Device:C
- removed C2: 10uF, Capacitor_SMD:C_1206_3216Metric_Pad1.33x1.80mm_HandSolder, symbol Device:C
- removed J12, J16, J3, J8: 10018783-10101TLF, avid_footprints:AMPHENOL_10018783-10101TLF, symbol 10018783-10101TLF:10018783-10101TLF
- removed J19: 901362104, avid_footprints:901362104, symbol avid_symbols:901362104
- removed J27, J28, J29, J30, J31: 901362103, 901362103, symbol avid_symbols:901362103
- removed R16, R17: CAY16-221J4LF, avid_footprints:CAY16_221J4LF, symbol CAY16_221J4LF:CAY16-221J4LF
- removed R18: 10k, Resistor_SMD:R_1206_3216Metric_Pad1.30x1.75mm_HandSolder, symbol Device:R
- removed U2: INA260AIPWR, PW0016A_N, symbol INA260AIPWR:INA260AIPWR
- removed U5: YC248-JR-0710KL, avid_footprints:RES_YC248_4X1P6_YAG, symbol avid_symbols:YC248-JR-0710KL
- removed U6: PCA9685PW, SOT361-1_NXP, symbol PCA9685PW:PCA9685PW
- added C19, C20, C21, C22: ECA-2AHG471, avid_footprints:ECA_2AHG471, symbol avid_symbols:ECA-2AHG471
- added J12, J16, J3, J8: 10018783-10101TLF, avid_footprints:AMPHENOL_10018783-10101TLF, symbol avid_symbols:10018783-10101TLF
- added R32: 4.7k, Resistor_SMD:R_1206_3216Metric_Pad1.30x1.75mm_HandSolder, symbol Device:R
- added R33, R34: 22k, Resistor_SMD:R_1206_3216Metric_Pad1.30x1.75mm_HandSolder, symbol Device:R
- J5: footprint DT1308PB -> avid_footprints:DT1308PB
Connections:
- net 24V: now also J5.8, J12.B20 (+VLOG), J16.B20 (+VLOG), J3.B20 (+VLOG), J8.B20 (+VLOG); no longer J5.2
- net BATT+: now also J5.1, J5.2, C19.1, C20.1, C21.1, C22.1, J12.A21 (+VMOT), J12.A22 (+VMOT), J12.B21 (+VMOT), J12.B22 (+VMOT), J16.A21 (+VMOT), J16.A22 (+VMOT), J16.B21 (+VMOT), J16.B22 (+VMOT), J3.A21 (+VMOT), J3.A22 (+VMOT), J3.B21 (+VMOT), J3.B22 (+VMOT), J8.A21 (+VMOT), J8.A22 (+VMOT), J8.B21 (+VMOT), J8.B22 (+VMOT); no longer J5.3, J5.4, J5.5
- net CLAMP_NC: no longer J20.1
- net DVR_+5VOUT_2: no longer J6.8, J7.2, J7.4
- net DVR_+5VOUT_3: no longer J10.8, J11.2, J11.4
- net DVR_+5VOUT_4: no longer J14.8, J15.2, J15.4
- net DVR_A-/SIN-/LH1_2: no longer J7.5
- net DVR_A-/SIN-/LH1_3: no longer J11.5
- net DVR_A/A+_2: no longer J6.1
- net DVR_A/A+_3: no longer J10.1
- net DVR_A/A+_4: no longer J14.1
- net DVR_A/SIN+_2: no longer J7.6
- net DVR_A/SIN+_3: no longer J11.6
- net DVR_B-/COS-/LH2_2: no longer J7.7
- net DVR_B-/COS-/LH2_3: no longer J11.7
- net DVR_B-/COS-/LH2_4: no longer J15.7
- net DVR_BR/B-_2: no longer J6.7
- net DVR_BR/B-_3: no longer J10.7
- net DVR_BR/B-_4: no longer J14.7
- net DVR_B/A-_2: no longer J6.6
- net DVR_B/A-_3: no longer J10.6
- net DVR_B/A-_4: no longer J14.6
- net DVR_B/COS+_2: no longer J7.8
- net DVR_B/COS+_3: no longer J11.8
- net DVR_B/COS+_4: no longer J15.8
- net DVR_C/B+_2: no longer J6.2
- net DVR_C/B+_3: no longer J10.2
- net DVR_C/B+_4: no longer J14.2
- net DVR_HALL1_2: no longer J6.3
- net DVR_HALL1_3: no longer J10.3
- net DVR_HALL1_4: no longer J14.3
- net DVR_HALL2_2: no longer J6.4
- net DVR_HALL2_3: no longer J10.4
- net DVR_HALL2_4: no longer J14.4
- net DVR_HALL3_2: no longer J6.5
- net DVR_HALL3_3: no longer J10.5
- net DVR_HALL3_4: no longer J14.5
- net DVR_Z+_2: no longer J7.10
- net DVR_Z+_3: no longer J11.10
- net DVR_Z+_4: no longer J15.10
- net DVR_Z-/LH3_2: no longer J7.9
- net DVR_Z-/LH3_3: no longer J11.9
- net DVR_Z-/LH3_4: no longer J15.9
- net GND: now also J20.1, J5.3, J5.4, J5.5, C19.2, C20.2, C21.2, C22.2, J12.A1 (GND), J12.A12 (GND), J12.A20 (GND), J12.A23 (GND), J12.A24 (GND), J12.B1 (GND), J12.B23 (GND), J12.B24 (GND), J12.B5 (GND), J12.B7 (AXISID1), J12.B8 (AXISID2), J16.A1 (GND), J16.A12 (GND), J16.A20 (GND), J16.A23 (GND), J16.A24 (GND), J16.B1 (GND), J16.B23 (GND), J16.B24 (GND), J16.B7 (AXISID1), J16.B8 (AXISID2), J3.A12 (GND), J3.A20 (GND), J3.A23 (GND), J3.A24 (GND), J3.B1 (GND), J3.B23 (GND), J3.B24 (GND), J3.B5 (GND), J3.B7 (AXISID1), J3.B8 (AXISID2), J8.A1 (GND), J8.A12 (GND), J8.A20 (GND), J8.A23 (GND), J8.A24 (GND), J8.B1 (GND), J8.B23 (GND), J8.B24 (GND), J8.B5 (GND), J8.B7 (AXISID1), J8.B8 (AXISID2), R32.2, R33.2; no longer J5.1, J5.8
- net DVR_+5VOUT_1 renamed D1_+5VOUT
- net D1_+5VOUT: now also J3.A11 (+5VOUT), J3.B11 (+5VOUT)
- net DVR_A-/SIN-/LH1_1 renamed D1_A-
- net D1_A-: now also J3.A14 (A/SIN+)
- net DVR_A-/SIN-/LH1_4 renamed D4_A-
- net D4_A-: now also J16.A14 (A/SIN+)
- net DVR_A/A+_1 renamed D1_A/A+
- net D1_A/A+: now also J3.B29 (A/A+), J3.B30 (A/A+), J3.B31 (A/A+), J3.B32 (A/A+)
- net DVR_A/SIN+_1 renamed D1_A+
- net D1_A+: now also J3.A13 (A-/SIN-/LH1)
- net DVR_A/SIN+_4 renamed D4_A+
- net D4_A+: now also J16.A13 (A-/SIN-/LH1)
- net DVR_B-/COS-/LH2_1 renamed D1_B-
- net D1_B-: now also J3.A15 (B-/COS-/LH2)
- net DVR_BR/B-_1 renamed D1_BR/B-
- net D1_BR/B-: now also J3.A25 (BR/B-), J3.A26 (BR/B-), J3.A27 (BR/B-), J3.A28 (BR/B-)
- net DVR_B/A-_1 renamed D1_B/A-
- net D1_B/A-: now also J3.A29 (B/A-), J3.A30 (B/A-), J3.A31 (B/A-), J3.A32 (B/A-)
- net DVR_B/COS+_1 renamed D1_B+
- net D1_B+: now also J3.A16 (B/COS+)
- net DVR_CAN_1_+ renamed CAN+
- net CAN+: now also J12.A19 (CAN-HI), J16.A19 (CAN-HI), J3.A19 (CAN-HI), J8.A19 (CAN-HI)
- net DVR_CAN_1_- renamed CAN-
- net CAN-: now also J12.B19 (CAN-LO), J16.B19 (CAN-LO), J3.B19 (CAN-LO), J8.B19 (CAN-LO)
- net DVR_C/B+_1 renamed D1_C/B+
- net D1_C/B+: now also J3.B25 (C/B+), J3.B26 (C/B+), J3.B27 (C/B+), J3.B28 (C/B+)
- net DVR_HALL1_1 renamed D1_HALL1
- net D1_HALL1: now also J3.A8 (HALL1)
- net DVR_HALL2_1 renamed D1_HALL2
- net D1_HALL2: now also J3.A9 (HALL2)
- net DVR_HALL3_1 renamed D1_HALL3
- net D1_HALL3: now also J3.A10 (HALL3)
- net DVR_Z+_1 renamed D1_Z+
- net D1_Z+: now also J3.A18 (Z+)
- net DVR_Z-/LH3_1 renamed D1_Z-
- net D1_Z-: now also J3.A17 (Z-/LH3)
- new net: J3.B6 (AXISID0), R32.1
- new net: J16.B6 (AXISID0), R34.2
- new net: J8.B6 (AXISID0), R33.1
- new net D2_+5VOUT: J6.8, J7.2, J7.4, J8.A11 (+5VOUT), J8.B11 (+5VOUT)
- new net D2_A+: J7.6, J8.A13 (A-/SIN-/LH1)
- new net D2_A-: J7.5, J8.A14 (A/SIN+)
- new net D2_A/A+: J6.1, J8.B29 (A/A+), J8.B30 (A/A+), J8.B31 (A/A+), J8.B32 (A/A+)
- new net D2_B+: J7.8, J8.A16 (B/COS+)
- new net D2_B-: J7.7, J8.A15 (B-/COS-/LH2)
- new net D2_BR/B-: J6.7, J8.A25 (BR/B-), J8.A26 (BR/B-), J8.A27 (BR/B-), J8.A28 (BR/B-)
- new net D2_B/A-: J6.6, J8.A29 (B/A-), J8.A30 (B/A-), J8.A31 (B/A-), J8.A32 (B/A-)
- new net D2_C/B+: J6.2, J8.B25 (C/B+), J8.B26 (C/B+), J8.B27 (C/B+), J8.B28 (C/B+)
- new net D2_HALL1: J6.3, J8.A8 (HALL1)
- new net D2_HALL2: J6.4, J8.A9 (HALL2)
- new net D2_HALL3: J6.5, J8.A10 (HALL3)
- new net D2_Z+: J7.10, J8.A18 (Z+)
- new net D2_Z-: J7.9, J8.A17 (Z-/LH3)
- new net D3_+5VOUT: J10.8, J11.2, J11.4, J12.A11 (+5VOUT), J12.B11 (+5VOUT)
- new net D3_A+: J11.6, J12.A13 (A-/SIN-/LH1)
- new net D3_A-: J11.5, J12.A14 (A/SIN+)
- new net D3_A/A+: J10.1, J12.B29 (A/A+), J12.B30 (A/A+), J12.B31 (A/A+), J12.B32 (A/A+)
- new net D3_B+: J11.8, J12.A16 (B/COS+)
- new net D3_B-: J11.7, J12.A15 (B-/COS-/LH2)
- new net D3_BR/B-: J10.7, J12.A25 (BR/B-), J12.A26 (BR/B-), J12.A27 (BR/B-), J12.A28 (BR/B-)
- new net D3_B/A-: J10.6, J12.A29 (B/A-), J12.A30 (B/A-), J12.A31 (B/A-), J12.A32 (B/A-)
- new net D3_C/B+: J10.2, J12.B25 (C/B+), J12.B26 (C/B+), J12.B27 (C/B+), J12.B28 (C/B+)
- new net D3_HALL1: J10.3, J12.A8 (HALL1)
- new net D3_HALL2: J10.4, J12.A9 (HALL2)
- new net D3_HALL3: J10.5, J12.A10 (HALL3)
- new net D3_Z+: J11.10, J12.A18 (Z+)
- new net D3_Z-: J11.9, J12.A17 (Z-/LH3)
- new net D4_+5VOUT: J14.8, J15.2, J15.4, J16.A11 (+5VOUT), J16.B11 (+5VOUT), R34.1
- new net D4_A/A+: J14.1, J16.B29 (A/A+), J16.B30 (A/A+), J16.B31 (A/A+), J16.B32 (A/A+)
- new net D4_B+: J15.8, J16.A16 (B/COS+)
- new net D4_B-: J15.7, J16.A15 (B-/COS-/LH2)
- new net D4_BR/B-: J14.7, J16.A25 (BR/B-), J16.A26 (BR/B-), J16.A27 (BR/B-), J16.A28 (BR/B-)
- new net D4_B/A-: J14.6, J16.A29 (B/A-), J16.A30 (B/A-), J16.A31 (B/A-), J16.A32 (B/A-)
- new net D4_C/B+: J14.2, J16.B25 (C/B+), J16.B26 (C/B+), J16.B27 (C/B+), J16.B28 (C/B+)
- new net D4_HALL1: J14.3, J16.A8 (HALL1)
- new net D4_HALL2: J14.4, J16.A9 (HALL2)
- new net D4_HALL3: J14.5, J16.A10 (HALL3)
- new net D4_Z+: J15.10, J16.A18 (Z+)
- new net D4_Z-: J15.9, J16.A17 (Z-/LH3)
Other:
- sheet CM4_HighSpeed ports: added USB2_+, USB2_-; removed USB2_N, USB2_P
- sheet USB2-HUB ports: added USB2_+, USB2_-; removed USB2_N, USB2_P
- note added: "1. GND 2. +5VOUT 3. GND 4. +5VOUT 5. A- 6. A+ 7. B- 8. B+ 9. Z- 10. Z+"
- note added: "ENC1: PHASE A - CAM_D0 - PH9 PHASE B - CAM_D1 - PH10 PHASE Z - CAM_D2 - PH11 ENC2: PHASE A - CAM_D3 - PH12 PHASE B - CAM_D4 - PH14 PHASE Z - CAM_D5 - PI4"
- note added: "INA260AIPWR"
- note added: "Motor Drivers (PRO-A04V36A-CAN) Following config 4 in the datasheet"
- note added: "OPENCAN Axis ID = 001 Axis ID 0 4.7k - GND Axis ID 1 GND Axis ID 2 GND"
- note added: "OPENCAN Axis ID = 002 Axis ID 0 22k - GND Axis ID 1 GND Axis ID 2 GND"
- note added: "OPENCAN Axis ID = 003 Axis ID 0 FLOATER!!! Axis ID 1 GND Axis ID 2 GND"
- note added: "OPENCAN Axis ID = 004 Axis ID 0 22k - 5V Axis ID 1 GND Axis ID 2 GND"
- note removed: "24V Monitor I2C Address: 100 1111 : 4F"
- note removed: "43045-1012 is the same part number as J2 on the PRO-A0xV36x-SA-CAN"
- note removed: "43045-1012 is the same part number as J3 on the PRO-A0xV36x-SA-CAN"
- note removed: "Motor Drivers (PRO-A04V36A-CAN)"
- note removed: "PCA9685 LED All Call Address (1110 000) and software reset (0000 0110) are active on start up (avoid these) Base Address: 0100 0000 : 40"
- note removed: "Servo Driver"
- note removed: "i2c input"
- moved on the sheet: IC2, J1, J18, J2, J6, LED1, Q1, R10, R11, R12, R13, R14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

Commit message: ordered power and control A4
Parts:
- added CR1: PMEG6020ER_115, avid_footprints:CFP3_SOD123W_NEX, symbol avid_symbols:PMEG6020ER_115
Connections:
- net 5V: now also CR1.2; no longer U1.J1_21 (VIN), U1.J1_32 (VIN), U1.J1_41 (VIN), U1.J1_48 (VIN)
- new net: CR1.1, U1.J1_21 (VIN), U1.J1_32 (VIN), U1.J1_41 (VIN), U1.J1_48 (VIN)
Changed lines of the file:
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@@
 	)
 	(junction
+		(at 151.13 44.45)
+		(diameter 0)
+		(color 0 0 0 0)
+	)
+	(junction
 		(at 25.4 317.5)
 		(diameter 0)
@@
 	)
 	(junction
+		(at 151.13 41.91)
+		(diameter 0)
+		(color 0 0 0 0)
+	)
+	(junction
+		(at 151.13 39.37)
+		(diameter 0)
+		(color 0 0 0 0)
+	)
+	(junction
 		(at 450.85 436.88)
 		(diameter 0)
@@
 	(wire
 		(pts
+			(xy 147.32 39.37) (xy 151.13 39.37)
+		)
+		(stroke
+			(width 0)
+			(type default)
+		)
+	)
+	(wire
+		(pts
+			(xy 135.89 39.37) (xy 137.16 39.37)
+		)
+		(stroke
+			(width 0)
+			(type default)
+		)
+	)
+	(wire
+		(pts
 			(xy 590.55 224.79) (xy 622.3 224.79)
 		)
@@
 	(wire
 		(pts
+			(xy 151.13 39.37) (xy 151.13 41.91)
+		)
+		(stroke
+			(width 0)
+			(type default)
+		)
+	)
+	(wire
+		(pts
 			(xy 193.04 226.06) (xy 189.23 226.06)
 		)
@@
 	(wire
 		(pts
+			(xy 151.13 41.91) (xy 151.13 44.45)
+		)
+		(stroke
+			(width 0)
+			(type default)
+		)
+	)
+	(wire
+		(pts
 			(xy 168.91 229.87) (xy 189.23 229.87)
 		)
@@
 	(wire
 		(pts
+			(xy 151.13 44.45) (xy 151.13 46.99)
+		)
+		(stroke
+			(width 0)
+			(type default)
+		)
+	)
+	(wire
+		(pts
 			(xy 582.93 345.44) (xy 599.44 345.44)
 		)
@@
 		)
 	)
+	(global_label "5V"
+		(shape input)
+		(at 135.89 39.37 180)
+		(fields_autoplaced yes)
+		(effects
+			(font
+				(size 1.27 1.27)
+			)
+			(justify right)
+		)
+		(property "Intersheetrefs" "${INTERSHEET_REFS}"
+			(at 130.6067 39.37 0)
+			(effects
+				(font
+					(size 1.27 1.27)
+				)
+				(justify right)
+				(hide yes)
+			)
+		)
+	)
 	(global_label "GND"
 		(shape input)
@@
 		)
 	)
-	(global_label "5V"
-		(shape input)
-		(at 151.13 44.45 180)
-		(fields_autoplaced yes)
-		(effects
-			(font
-				(size 1.27 1.27)
-			)
-			(justify right)
-		)
-		(property "Intersheetrefs" "${INTERSHEET_REFS}"
-			(at 145.8467 44.45 0)
-			(effects
-				(font
-					(size 1.27 1.27)
-				)
-				(justify right)
-				(hide yes)
-			)
-		)
-	)
 	(global_label "D4_B+"
 		(shape input)
@@
 		)
 	)
-	(global_label "5V"
-		(shape input)
-		(at 151.13 46.99 180)
-		(fields_autoplaced yes)
-		(effects
-			(font
-				(size 1.27 1.27)
-			)
-			(justify right)
-		)
-		(property "Intersheetrefs" "${INTERSHEET_REFS}"
-			(at 145.8467 46.99 0)
-			(effects
-				(font
-					(size 1.27 1.27)
-				)
-				(justify right)
-				(hide yes)
-			)
-		)
-	)
 	(global_label "D3_HALL1"
 		(shape input)
@@
 		)
 	)
-	(global_label "5V"
-		(shape input)
-		(at 151.13 39.37 180)
-		(fields_autoplaced yes)
-		(effects
-			(font
-				(size 1.27 1.27)
-			)
-			(justify right)
-		)
-		(property "Intersheetrefs" "${INTERSHEET_REFS}"
-			(at 145.8467 39.37 0)
-			(effects
-				(font
-					(size 1.27 1.27)
-				)
-				(justify right)
-				(hide yes)
-			)
-		)
-	)
 	(global_label "D4_+5VOUT"
 		(shape input)
@@
 		)
 	)
-	(global_label "5V"
-		(shape input)
-		(at 151.13 41.91 180)
-		(fields_autoplaced yes)
-		(effects
-			(font
-				(size 1.27 1.27)
-			)
-			(justify right)
-		)
-		(property "Intersheetrefs" "${INTERSHEET_REFS}"
-			(at 145.8467 41.91 0)
-			(effects
-				(font
-					(size 1.27 1.27)
-				)
-				(justify right)
-				(hide yes)
-			)
-		)
-	)
 	(global_label "DVR_OUT0_4"
 		(shape input)
@@
 					(unit 1)
 				)
+			)
+		)
+	)
+	(symbol
+		(lib_id "avid_symbols:PMEG6020ER_115")
+		(at 137.16 39.37 0)
+		(unit 1)
+		(exclude_from_sim no)
+		(in_bom yes)
+		(on_board yes)
+		(dnp no)
+		(fields_autoplaced yes)
+		(property "Reference" "CR1"
+			(at 142.24 33.02 0)
+			(effects
+				(font
+					(size 1.524 1.524)
+				)
+			)
+		)
+		(property "Value" "PMEG6020ER_115"
+			(at 142.24 35.56 0)
+			(effects
+				(font
+					(size 1.524 1.524)
+				)
+			)
+		)
+		(property "Footprint" "avid_footprints:CFP3_SOD123W_NEX"
+			(at 137.16 39.37 0)
+			(effects
+				(font
+					(size 1.27 1.27)
+					(italic yes)
+				)
+				(hide yes)
+			)
+		)
+		(property "Datasheet" "PMEG6020ER_115"
+			(at 137.16 39.37 0)
+			(effects
+				(font
+					(size 1.27 1.27)
+					(italic yes)
+				)
+				(hide yes)
+			)
+		)
+		(property "Description" ""
+			(at 137.16 39.37 0)
+			(effects
+				(font
+					(size 1.27 1.27)
+				)
+				(hide yes)
+			)
+		)
+		(pin "1"
+		)
+		(pin "2"
+		)
+		(instances
+			(project "GR-LRR-CONTROL"
+				(path "/7e750e3c-c787-4adb-8081-69356fc148e5"
+					(reference "CR1")
+					(unit 1)
+				)

Commit message: upload
Parts:
- removed R34: 22k, Resistor_SMD:R_1206_3216Metric_Pad1.30x1.75mm_HandSolder, symbol Device:R
- added R16: 22k, Resistor_SMD:R_1206_3216Metric_Pad1.30x1.75mm_HandSolder, symbol Device:R
- CR1: Part Number (none) -> PMEG6020ER_115
- IC1: Part Number (none) -> TJA1049T,118
- J1, J11, J15, J7: Part Number (none) -> 87833-1019
- J10, J14, J2, J6: Part Number (none) -> 430451000
- J12, J16, J3, J8: Part Number (none) -> 10018783-10101TLF
- J18: Part Number (none) -> 691137710002
- J20: Part Number (none) -> 901362102
- J21, J22: Part Number (none) -> 901362105
- J23, J24: Part Number (none) -> 901362104
- J25: value UT1 -> LED; Part Number (none) -> 901362104
- J26: value UT2 -> LED; Part Number (none) -> 901362104
- J5: Part Number (none) -> DT13-08PB
- R1, R2: Part Number (none) -> RNCS1206BKE10K0
- R10, R12: Part Number (none) -> YC164-JR-072KL
- R11, R14: value 10k 1/8W -> 10k
- R3, R31: value 120 -> 120 1/4W; Part Number (none) -> RT1206DRE07120RL
- R32: Part Number (none) -> RC1206JR-074K7L
- R33: Part Number (none) -> RC1206FR-0722KL
- R8: Part Number (none) -> RNCS1206BKE100K
- R9: value 10k 1/8w -> 10k; Part Number (none) -> RNCS1206BKE10K0
Connections:
- net D4_+5VOUT: now also R16.1
- net GND: now also IC1.8 (STB)
- net at J16.B6 (AXISID0): now also R16.2
Other:
- note added: "H7 Connector: DF40HC(3.5)-80DS-0.4V(51)"
- note added: "STAND BY MUST BE PULLED LOW"
- note added: "Zigbee Connector: 2RS1-10-G"
- moved on the sheet: R1
