File: GR-LRR-CONTROL/USB2-HUB.kicad_sch (KiCad schematic)
At the start: 32 parts, among them J38 690-008-221-904, J7 USB_OTG, J8 690-008-221-904, U10 AP22653W6, U7 FSUSB42MUX, U8 USB2514B-I/M2, U9 TPD4EUSB30, Y1 24MHz

Commit message: finished routing
Connections:
- net USB2_N renamed USB2_-
- net USB2_P renamed USB2_+
Changed lines of the file:
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@@
 		)
 	)
-	(hierarchical_label "USB2_N"
+	(hierarchical_label "USB2_-"
 		(shape bidirectional)
 		(at 27.94 64.77 180)
@@
 		)
 	)
-	(hierarchical_label "USB2_P"
+	(hierarchical_label "USB2_+"
 		(shape bidirectional)
 		(at 27.94 62.23 180)

Commit message: upload
Parts:
- C10, C11, C12, C13, C14, C9: Field6 RM EMK105 B7104KV-F -> (none); Part Number (none) -> RM EMK105 B7104KV-F
- C15, C17, C18, C19, C20, C7, C8: Field6 GRM21BR71A106KA73L -> (none); Part Number (none) -> GRM21BR71A106KA73L
- C16: Field5 667-EEF-CX0J101R -> (none); Part Number (none) -> EEF-CX0J101R
- C5, C6: Field6 GJM1555C1H270JB01D -> (none); Part Number (none) -> GJM1555C1H270JB01D
- J38, J8: Field8 UCON00727 -> (none); Part Number (none) -> 0672984090
- J7: Field5 609-4050-2-ND -> (none); Part Number (none) -> 10103594-0001LF
- R29, R30: Part Number (none) -> RC0402FR-072K2L
- R31, R40, R41, R47: Part Number (none) -> CRCW040236K0FKED
- R46: Part Number (none) -> RC0402FR-0712KL
- R48: Field6 MCR01MZPF1502 -> (none); Part Number (none) -> CRCW040215K0FKED
- U10: Field6 AP22653W6 -> (none); Part Number (none) -> AP22653W6
- U7: Field6 FSUSB42MUX -> (none); Part Number (none) -> FSUSB42MUX
- U8: Field6 USB2514B-I/M2 -> (none); Part Number (none) -> USB2514B-I/M2
- U9: Field6 CDDFN10-3324P-13 -> (none); Part Number (none) -> CDDFN10-3324P
- Y1: Field6 X24M000000S128 -> (none); Part Number (none) -> QCS24.0000F18B23M
Changed lines of the file:
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@@
 			)
 		)
-		(property "Field8" "UCON00727"
+		(property "Part Number" "0672984090"
 			(at 207.01 125.73 0)
 			(effects
@@
 			)
 		)
-		(property "Field5" "609-4050-2-ND"
+		(property "Part Number" "10103594-0001LF"
 			(at 128.27 39.37 0)
 			(effects
@@
 			)
 		)
+		(property "Part Number" "RC0402FR-072K2L"
+			(at 40.64 45.72 0)
+			(effects
+				(font
+					(size 1.27 1.27)
+				)
+				(hide yes)
+			)
+		)
 		(pin "1"
 		)
@@
 			)
 		)
-		(property "Field6" "GRM21BR71A106KA73L"
+		(property "Part Number" "GRM21BR71A106KA73L"
 			(at 243.84 83.82 0)
 			(effects
@@
 			)
 		)
-		(property "Field6" "GRM21BR71A106KA73L"
+		(property "Part Number" "GRM21BR71A106KA73L"
 			(at 254 83.82 0)
 			(effects
@@
 			)
 		)
-		(property "Field6" "GRM21BR71A106KA73L"
+		(property "Part Number" "GRM21BR71A106KA73L"
 			(at 264.16 83.82 0)
 			(effects
@@
 			)
 		)
-		(property "Field6" "GRM21BR71A106KA73L"
+		(property "Part Number" "GRM21BR71A106KA73L"
 			(at 274.32 83.82 0)
 			(effects
@@
 			)
 		)
+		(property "Part Number" "RC0402FR-072K2L"
+			(at 33.02 72.39 0)
+			(effects
+				(font
+					(size 1.27 1.27)
+				)
+				(hide yes)
+			)
+		)
 		(pin "1"
 		)
@@
 			)
 		)
-		(property "Field6" "AP22653W6"
+		(property "Part Number" "AP22653W6"
 			(at 203.2 80.01 0)
 			(effects
@@
 			)
 		)
-		(property "Field6" "USB2514B-I/M2"
+		(property "Part Number" "USB2514B-I/M2"
 			(at 123.19 111.76 0)
 			(effects
@@
 			)
 		)
+		(property "Part Number" "CRCW040236K0FKED"
+			(at 83.82 146.05 90)
+			(effects
+				(font
+					(size 1.27 1.27)
+				)
+				(hide yes)
+			)
+		)
 		(pin "1"
 		)
@@
 			)
 		)
+		(property "Part Number" "CRCW040236K0FKED"
+			(at 76.2 146.05 90)
+			(effects
+				(font
+					(size 1.27 1.27)
+				)
+				(hide yes)
+			)
+		)
 		(pin "1"
 		)
@@
 			)
 		)
+		(property "Part Number" "CRCW040236K0FKED"
+			(at 68.58 146.05 90)
+			(effects
+				(font
+					(size 1.27 1.27)
+				)
+				(hide yes)
+			)
+		)
 		(pin "1"
 		)
@@
 			)
 		)
-		(property "Field6" "MCR01MZPF1502"
+		(property "Part Number" "CRCW040215K0FKED"
 			(at 222.25 80.01 0)
 			(effects
@@
 			)
 		)
-		(property "Field6" "FSUSB42MUX"
+		(property "Part Number" "FSUSB42MUX"
 			(at 52.07 72.39 0)
 			(effects
@@
 			)
 		)
+		(property "Part Number" "RC0402FR-0712KL "
+			(at 86.36 109.22 90)
+			(effects
+				(font
+					(size 1.27 1.27)
+				)
+				(hide yes)
+			)
+		)
 		(pin "1"
 		)
@@
 			)
 		)
+		(property "Part Number" "CRCW040236K0FKED"
+			(at 91.44 146.05 90)
+			(effects
+				(font
+					(size 1.27 1.27)
+				)
+				(hide yes)
+			)
+		)
 		(pin "1"
 		)
@@
 			)
 		)
-		(property "Field6" "RM EMK105 B7104KV-F"
+		(property "Part Number" "RM EMK105 B7104KV-F"
 			(at 116.84 168.91 0)
 			(effects
@@
 			)
 		)
-		(property "Field6" "RM EMK105 B7104KV-F"
+		(property "Part Number" "RM EMK105 B7104KV-F"
 			(at 128.27 168.91 0)
 			(effects
@@
 			)
 		)
-		(property "Field6" "RM EMK105 B7104KV-F"
+		(property "Part Number" "RM EMK105 B7104KV-F"
 			(at 138.43 168.91 0)
 			(effects
@@
 			)
 		)
-		(property "Field6" "RM EMK105 B7104KV-F"
+		(property "Part Number" "RM EMK105 B7104KV-F"
 			(at 93.218 168.91 0)
 			(effects
@@
 			)
 		)
-		(property "Field6" "GRM21BR71A106KA73L"
+		(property "Part Number" "GRM21BR71A106KA73L"
 			(at 74.93 168.91 0)
 			(effects
@@
 			)
 		)
-		(property "Field6" "GRM21BR71A106KA73L"
+		(property "Part Number" "GRM21BR71A106KA73L"
 			(at 84.074 168.91 0)
 			(effects
@@
 			)
 		)
-		(property "Field6" "X24M000000S128"
+		(property "Part Number" "QCS24.0000F18B23M"
 			(at 48.26 125.73 0)
 			(effects
@@
 			)
 		)
-		(property "Field6" "GJM1555C1H270JB01D"
+		(property "Part Number" "GJM1555C1H270JB01D"
 			(at 36.83 130.81 0)
 			(effects
@@
 			)
 		)
-		(property "Field6" "GJM1555C1H270JB01D"
+		(property "Part Number" "GJM1555C1H270JB01D"
 			(at 57.15 130.81 0)
 			(effects
@@
 			)
 		)
-		(property "Field6" "RM EMK105 B7104KV-F"
+		(property "Part Number" "RM EMK105 B7104KV-F"
 			(at 103.378 168.91 0)
 			(effects
@@
 			)
 		)
-		(property "Field6" "RM EMK105 B7104KV-F"
+		(property "Part Number" "RM EMK105 B7104KV-F"
 			(at 148.844 168.91 0)
 			(effects
@@
 			)
 		)
-		(property "Field6" "GRM21BR71A106KA73L"
+		(property "Part Number" "GRM21BR71A106KA73L"
 			(at 172.72 82.55 0)
 			(effects
@@
 			)
 		)
-		(property "Field6" "CDDFN10-3324P-13"
+		(property "Part Number" "CDDFN10-3324P"
 			(at 201.93 43.18 0)
 			(effects
@@
 			)
 		)
-		(property "Field5" "667-EEF-CX0J101R"
+		(property "Part Number" "EEF-CX0J101R"
 			(at 230.378 83.82 0)
 			(effects
@@
 			)
 		)
-		(property "Field8" "UCON00727"
+		(property "Part Number" "0672984090"
 			(at 255.27 124.46 0)
 			(effects
