File: GR-LRR-POWER/GR-LRR-POWER.kicad_pcb (KiCad board)
At the start: 2 copper layers, 213.7 x 137.6 mm, 50 parts, among them J1 DT13-08PB, J2 DT13-08PB, J3 Switch, J4 Switch, J5 Switch, U1 SIS434DN-T1-GE3, U2 SIS434DN-T1-GE3, U3 LTC4365CTS8-TRMPBF, U4 696108003002, U5 696108003002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

Commit message: purchasing A3 power
Parts:
- removed C2: 33uF, 50V Tant, avid_footprints:CAPMP7.6X4.3_4.3N_KEM-L
- removed C3: 220uF, 50V, Elec, avid_footprints:U2-R_NCH-L
- removed D1: SMCJ40A, avid_footprints:DIOM7959X262N
- removed J4, J5: Switch, avid_footprints:212520-1002
- removed L1: 12uF, 10.5A, Inductor_SMD:L_Coilcraft_XAL8080-XXX
- removed U4: 696108003002, avid_footprints:WR-FSH_THT_2
- added H2: MountingHole_Pad, MountingHole:MountingHole_3mm_Pad_Via, F.Cu at (177.5, 72.2)
- J3: value Switch -> 691137710002; footprint avid_footprints:212520-1002 -> avid_footprints:691137710002
- moved J3 29.3 mm to (91.8, 108.5)
- moved U3 28.4 mm to (110.9, 103.5)
- moved R1 26.6 mm to (104.0, 102.9)
- moved R2 26.6 mm to (100.2, 102.9)
- moved R3 26.6 mm to (100.2, 108.0)
- moved R4 26.6 mm to (100.2, 113.0)
- moved C1 18.3 mm to (116.1, 112.0), turned to 180 degrees
- moved U1 12.0 mm to (109.0, 96.2)
- moved U2 12.0 mm to (113.6, 96.2)
- moved LED1 11.3 mm to (220.9, 137.0)
- moved R5 11.3 mm to (220.9, 131.7)
Connections:
- C1 pad 1: Net-(U3-VOUT) -> BATT+
- J2 pad 1: BG -> BATT+
- J2 pad 2: 24V -> BATT+
- J2 pad 3: 18V -> BG
- J2 pad 4: 18V -> BG
- J2 pad 5: BATT+ -> BG
- J2 pad 8: BG -> 24V
- J3 pad 1: Net-(U3-VOUT) -> SHDN_SW
- J3 pad 2: BATT+ -> BG
- R1 pad 2: Net-(U3-*SHDN) -> SHDN_SW
- R6 pad 2: 18V -> BATT+
- U2 pad 5: Net-(U3-VOUT) -> BATT+
- U2 pad 6: Net-(U3-VOUT) -> BATT+
- U2 pad 7: Net-(U3-VOUT) -> BATT+
- U2 pad 8: Net-(U3-VOUT) -> BATT+
- U3 pad 5: Net-(U3-*SHDN) -> SHDN_SW
- U3 pad 7: Net-(U3-VOUT) -> BATT+
Routing:
- net BATT+: track 82.8 -> 7.60 mm
- net 24V: track 67.5 -> 104.4 mm
- net SHDN_SW: track 0.00 -> 25.2 mm, vias 0 -> 2
- net Net-(U1-G): track 0.00 -> 15.4 mm, vias 0 -> 2
- net BG: track 228.9 -> 243.0 mm
- net Net-(U3-OV): track 0.00 -> 13.6 mm
- net Net-(U3-UV): track 0.00 -> 11.8 mm
- net 5V: track 132.1 -> 143.6 mm
- net 3.3V: track 200.5 -> 206.7 mm
- net BV: track 0.00 -> 6.17 mm
- removed copper zone on F.Cu, net 18V
- removed copper zone on F.Cu, net Net-(C2-Pad1)
- removed copper zone on F.Cu, net Net-(U3-VOUT)
Other:
- board text added: "1. BATT 2. BATT 3. GND 4. GND"
- board text added: "8. 24V 7. 5V 6. 3.3V 5. GND"
- board text added: "GR-LRR-POWER 05-09-2024 A3"
- board text added: "PINS 1-4 BV PINS 5-8 BGND"
- board text added: "SHDN GND"
- board text removed: "1. GND 2. 24V 3. 18V 4. 18V"
- board text removed: "8. GND 7. 5V 6. 3.3V 5. Batt"

Commit message: ordered power and control A4
Parts:
- added R10: 168, Resistor_SMD:R_1206_3216Metric_Pad1.30x1.75mm_HandSolder, B.Cu at (198.6, 132.9)
- added R11: 168, Resistor_SMD:R_1206_3216Metric_Pad1.30x1.75mm_HandSolder, B.Cu at (194.5, 182.4)
- added R9: 168, Resistor_SMD:R_1206_3216Metric_Pad1.30x1.75mm_HandSolder, B.Cu at (196.7, 158.6)
- moved C1 2.95 mm to (116.1, 115.0)
- moved J1 2.95 mm to (104.9, 88.5)
- moved J3 2.95 mm to (91.8, 111.5)
- moved R3 2.95 mm to (100.2, 110.9)
- moved R4 2.95 mm to (100.2, 115.9)
- moved U1 2.95 mm to (109.0, 99.2)
- moved U2 2.95 mm to (113.6, 99.1)
- moved U3 2.95 mm to (110.9, 106.5)
- moved R1 2.95 mm to (104.0, 105.8)
- moved R2 2.95 mm to (100.2, 105.8)
- moved J2 2.93 mm to (225.0, 88.5)
Connections:
- PS1 pad 6: unconnected-(PS1-OUTPUT_TRIM-Pad6) -> Net-(PS1-OUTPUT_TRIM)
- PS1 pad 7: unconnected-(PS1-+SENSE-Pad7) -> Net-(PS1-+SENSE)
- PS2 pad 6: unconnected-(PS2-OUTPUT_TRIM-Pad6) -> Net-(PS2-OUTPUT_TRIM)
- PS2 pad 7: unconnected-(PS2-+SENSE-Pad7) -> Net-(PS2-+SENSE)
- PS3 pad 4: unconnected-(PS3-OUTPUT_TRIM-Pad4) -> Net-(PS3-OUTPUT_TRIM)
Routing:
- net 3.3V: track 206.7 -> 196.8 mm
- net 5V: track 143.6 -> 138.7 mm
- net Net-(PS1-OUTPUT_TRIM): track 0.00 -> 4.71 mm
- net Net-(PS2-+SENSE): track 0.00 -> 4.63 mm
- net Net-(PS1-+SENSE): track 0.00 -> 4.63 mm
- net BG: track 243.0 -> 247.5 mm
- net Net-(PS2-OUTPUT_TRIM): track 0.00 -> 4.50 mm
- net Net-(PS3-OUTPUT_TRIM): track 0.00 -> 2.56 mm
- net 24V: track 104.4 -> 103.3 mm
Other:
- board text added: "GR-LRR-POWER-05-12-2024-A4"
- board text removed: "GR-LRR-POWER 05-09-2024 A3"

Commit message: upload
Connections:
- PS3 pad 2: unconnected-(PS3--VIN-Pad2) -> BG
- PS3 pad 6: BG -> unconnected-(PS3-ON/OFF_CONTROL-Pad6)
Routing:
- net BG: track 247.5 -> 237.9 mm
Changed lines of the file:
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@@
 	(net 26 "unconnected-(PS2--SENSE-Pad5)")
 	(net 27 "Net-(PS3-OUTPUT_TRIM)")
-	(net 28 "unconnected-(PS3--VIN-Pad2)")
+	(net 28 "unconnected-(PS3-ON{slash}OFF_CONTROL-Pad6)")
 	(net 29 "unconnected-(J1-PadMH3)")
 	(net 30 "unconnected-(J1-PadMH2)")
@@
 			)
 		)
+		(property "Part Number" "SIS434DN-T1-GE3"
+			(at 0 0 180)
+			(unlocked yes)
+			(layer "F.Fab")
+			(hide yes)
+			(effects
+				(font
+					(size 1 1)
+					(thickness 0.15)
+				)
+			)
+		)
 		(property ki_fp_filters "MOSFET_4DN-T1-E3_VIS")
 		(sheetname "Root")
@@
 			)
 		)
-		(property "Part Number" "T521X336M050ATE075"
+		(property "Part Number" "T521X336M050ATE050"
 			(at 0 0 -90)
 			(unlocked yes)
@@
 			)
 		)
+		(property "Part Number" "696108003002"
+			(at 0 0 0)
+			(unlocked yes)
+			(layer "F.Fab")
+			(hide yes)
+			(effects
+				(font
+					(size 1 1)
+					(thickness 0.15)
+				)
+			)
+		)
 		(sheetname "Root")
 		(sheetfile "GR-LRR-POWER.kicad_sch")
@@
 			)
 		)
+		(property "Part Number" "UWT1H221MNL1GS"
+			(at 0 0 -90)
+			(unlocked yes)
+			(layer "F.Fab")
+			(hide yes)
+			(effects
+				(font
+					(size 1 1)
+					(thickness 0.15)
+				)
+			)
+		)
+		(property "Field6" ""
+			(at 0 0 -90)
+			(unlocked yes)
+			(layer "F.Fab")
+			(hide yes)
+			(effects
+				(font
+					(size 1 1)
+					(thickness 0.15)
+				)
+			)
+		)
 		(property ki_fp_filters "U2-R_NCH U2-R_NCH-M U2-R_NCH-L")
 		(sheetname "Root")
@@
 			(layers "*.Cu" "*.Mask")
 			(remove_unused_layers no)
-			(net 28 "unconnected-(PS3--VIN-Pad2)")
+			(net 5 "BG")
 			(pinfunction "-VIN")
 			(pintype "passive")
@@
 			(layers "*.Cu" "*.Mask")
 			(remove_unused_layers no)
-			(net 5 "BG")
+			(net 28 "unconnected-(PS3-ON{slash}OFF_CONTROL-Pad6)")
 			(pinfunction "ON/OFF_CONTROL")
 			(pintype "passive")
@@
 			)
 		)
+		(property "Part Number" "UWS-24_2-Q12P-C"
+			(at 0 0 0)
+			(unlocked yes)
+			(layer "F.Fab")
+			(hide yes)
+			(effects
+				(font
+					(size 1 1)
+					(thickness 0.15)
+				)
+			)
+		)
 		(sheetname "Root")
 		(sheetfile "GR-LRR-POWER.kicad_sch")
@@
 			)
 		)
+		(property "Part Number" "UWS-510-Q12P-C"
+			(at 0 0 0)
+			(unlocked yes)
+			(layer "F.Fab")
+			(hide yes)
+			(effects
+				(font
+					(size 1 1)
+					(thickness 0.15)
+				)
+			)
+		)
 		(sheetname "Root")
 		(sheetfile "GR-LRR-POWER.kicad_sch")
@@
 			)
 		)
-		(property "Part Number" "T521X336M050ATE075"
+		(property "Part Number" "T521X336M050ATE050"
 			(at 0 0 -90)
 			(unlocked yes)
@@
 			)
 		)
+		(property "Part Number" "DT13-08PB"
+			(at 0 0 90)
+			(unlocked yes)
+			(layer "F.Fab")
+			(hide yes)
+			(effects
+				(font
+					(size 1 1)
+					(thickness 0.15)
+				)
+			)
+		)
 		(sheetname "Root")
 		(sheetfile "GR-LRR-POWER.kicad_sch")
@@
 			)
 		)
+		(property "Part Number" "50ZLH100MEFC8X11.5"
+			(at 0 0 180)
+			(unlocked yes)
+			(layer "F.Fab")
+			(hide yes)
+			(effects
+				(font
+					(size 1 1)
+					(thickness 0.15)
+				)
+			)
+		)
 		(property ki_fp_filters "CAP_YX_8X11P5_RUB")
 		(sheetname "Root")
@@
 			)
 		)
+		(property "Part Number" "691137710002"
+			(at 0 0 -90)
+			(unlocked yes)
+			(layer "F.Fab")
+			(hide yes)
+			(effects
+				(font
+					(size 1 1)
+					(thickness 0.15)
+				)
+			)
+		)
 		(property ki_fp_filters "CONN2_710002_WRE")
 		(sheetname "Root")
@@
 			)
 		)
+		(property "Part Number" "UWT1H221MNL1GS"
+			(at 0 0 -90)
+			(unlocked yes)
+			(layer "F.Fab")
+			(hide yes)
+			(effects
+				(font
+					(size 1 1)
+					(thickness 0.15)
+				)
+			)
+		)
 		(property ki_fp_filters "U2-R_NCH U2-R_NCH-M U2-R_NCH-L")
 		(sheetname "Root")
@@
 			)
 		)
+		(property "Part Number" "SIS434DN-T1-GE3"
+			(at 0 0 0)
+			(unlocked yes)
+			(layer "F.Fab")
+			(hide yes)
+			(effects
+				(font
+					(size 1 1)
+					(thickness 0.15)
+				)
+			)
+		)
 		(property ki_fp_filters "MOSFET_4DN-T1-E3_VIS")
 		(sheetname "Root")
@@
 			)
 		)
+		(property "Part Number" "UWT1H221MNL1GS"
+			(at 0 0 -90)
+			(unlocked yes)
+			(layer "F.Fab")
+			(hide yes)
+			(effects
+				(font
+					(size 1 1)
+					(thickness 0.15)
+				)
+			)
+		)
 		(property ki_fp_filters "U2-R_NCH U2-R_NCH-M U2-R_NCH-L")
 		(sheetname "Root")
@@
 			)
 		)
-		(property "Part Number" "T521X336M050ATE075"
+		(property "Part Number" "T521X336M050ATE050"
 			(at 0 0 -90)
 			(unlocked yes)
@@
 			)
 		)
+		(property "Part Number" "LTC4365CTS8-TRMPBF"
+			(at 0 0 0)
+			(unlocked yes)
+			(layer "F.Fab")
+			(hide yes)
+			(effects
+				(font
+					(size 1 1)
+					(thickness 0.15)
+				)
+			)
+		)
 		(property ki_fp_filters "TSOT-23_TS8_LIT TSOT-23_TS8_LIT-M TSOT-23_TS8_LIT-L")
 		(sheetname "Root")
@@
 		(tags "resistor handsolder")
 		(property "Reference" "R9"
-			(at 0 1.82 270)
+			(at 0 1.82 -90)
 			(layer "B.SilkS")
 			(effects
@@
 		)
 		(property "Value" "168"
-			(at 0 -1.82 270)
+			(at 0 -1.82 -90)
 			(layer "B.Fab")
 			(effects
@@
 		)
 		(fp_text user "${REFERENCE}"
-			(at 0 0 270)
+			(at 0 0 -90)
 			(layer "B.Fab")
 			(effects
@@
 		(tags "resistor handsolder")
 		(property "Reference" "R11"
-			(at 0 1.82 270)
+			(at 0 1.82 -90)
 			(layer "B.SilkS")
 			(effects
@@
 		)
 		(property "Value" "168"
-			(at 0 -1.82 270)
+			(at 0 -1.82 -90)
 			(layer "B.Fab")
 			(effects
@@
 		)
 		(fp_text user "${REFERENCE}"
-			(at 0 0 270)
+			(at 0 0 -90)
 			(layer "B.Fab")
 			(effects
@@
 		(tags "resistor handsolder")
 		(property "Reference" "R10"
-			(at 0 1.82 270)
+			(at 0 1.82 -90)
 			(layer "B.SilkS")
 			(effects
@@
 		)
 		(property "Value" "168"
-			(at 0 -1.82 270)
+			(at 0 -1.82 -90)
 			(layer "B.Fab")
 			(effects
@@
 		)
 		(fp_text user "${REFERENCE}"
-			(at 0 0 270)
+			(at 0 0 -90)
 			(layer "B.Fab")
 			(effects
@@
 		(width 2)
 		(layer "F.Cu")
-		(net 5)
-	)
-	(segment
-		(start 167.418645 183.116355)
-		(end 174.195 176.34)
-		(width 2)
-		(layer "F.Cu")
